File: kicad/imu-board/imu-board.kicad_sch (KiCad schematic)
At the start: 7 parts, among them U1 ICM-45686, U2 BMI088

Commit message: [LIMA] imu-board: split the shared SPI bus into two independent buses
Peter's call: the IMUs stay on this separate PCB but connect to the host over
individual SPIs. The board previously put all three dies on one 3-wire bus with
three chip selects - a common-mode failure path that defeats the point of
carrying two independent IMUs.

Now one bus per chip:
  ICM-45686  ICM_SCLK / ICM_MOSI / ICM_MISO / ICM_CS
  BMI088     BMI_SCLK / BMI_MOSI / BMI_ACC_SDO / BMI_GYR_SDO
The only nets shared between the two chips are +3V3 and GND, confirmed by
per-pin net readback rather than read off the drawing.

The BMI088's accel and gyro share SCK and SDI physically, so one bus per DIE is
impossible for that part - one bus per chip is the real limit. Bosch's
reference topology ties SDO1 and SDO2 onto a single MISO; we deliberately do
not. Tying them reinstates the common-mode failure we just removed, and with
both pins typed Output it raises a genuine [pin_to_pin] ERC error about real
contention that only the chip-select protocol prevents. Suppressing that would
have left a standing error to mask the next one. Kept separate, the decision
moves to the host board, which can tie them or drive two peripherals.

Verified: per-pin nets on both parts correct; find_shorted_nets 0; PS tied to
GND so the BMI088 is in SPI mode (already correct); ERC 19 violations, all
expected with no host present - 5 pin_not_driven and 14 isolated_pin_label. The
pin_to_pin output conflict is gone.

Note: this edits another session's project. That session committed at 03a9fc6
and has been idle since 17:00 yesterday, so the working tree was not live.
Connections:
- removed net IMU_MISO: U1.1 (AP_SDO/AP_AD0), U2.10 (SDO2), U2.15 (SDO1)
- net IMU_MOSI renamed BMI_MOSI
- net BMI_MOSI: no longer U1.14 (AP_SDA/AP_SDIO/AP_SDI)
- net IMU_SCLK renamed BMI_SCLK
- net BMI_SCLK: no longer U1.13 (AP_SCL/AP_SCLK)
- new net BMI_ACC_SDO: U2.15 (SDO1)
- new net BMI_GYR_SDO: U2.10 (SDO2)
- new net ICM_MISO: U1.1 (AP_SDO/AP_AD0)
- new net ICM_MOSI: U1.14 (AP_SDA/AP_SDIO/AP_SDI)
- new net ICM_SCLK: U1.13 (AP_SCL/AP_SCLK)
Changed lines of the file:
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@@
-		)
-	)
-	(label "IMU_SCLK"
-		(at 77.47 102.87 180)
-		(effects
-			(font
-				(size 1.27 1.27)
-			)
-			(justify right bottom)
-		)
-	)
-	(label "IMU_MOSI"
-		(at 77.47 105.41 180)
-		(effects
-			(font
-				(size 1.27 1.27)
-			)
-			(justify right bottom)
-		)
-	)
-	(label "IMU_MISO"
-		(at 77.47 107.95 180)
-		(effects
-			(font
-				(size 1.27 1.27)
-			)
-			(justify right bottom)
 		)
 	)
@@
 		)
 	)
-	(label "IMU_SCLK"
-		(at 264.16 107.95 180)
-		(effects
-			(font
-				(size 1.27 1.27)
-			)
-			(justify right bottom)
-		)
-	)
-	(label "IMU_MOSI"
-		(at 264.16 110.49 180)
-		(effects
-			(font
-				(size 1.27 1.27)
-			)
-			(justify right bottom)
-		)
-	)
-	(label "IMU_MISO"
-		(at 264.16 113.03 180)
-		(effects
-			(font
-				(size 1.27 1.27)
-			)
-			(justify right bottom)
-		)
-	)
-	(label "IMU_MISO"
-		(at 264.16 115.57 180)
-		(effects
-			(font
-				(size 1.27 1.27)
-			)
-			(justify right bottom)
-		)
-	)
 	(label "BMI_ACC_CS"
 		(at 264.16 102.87 180)
@@
 			)
 			(justify left bottom)
+		)
+	)
+	(label "ICM_SCLK"
+		(at 77.47 102.87 180)
+		(effects
+			(font
+				(size 1.27 1.27)
+			)
+			(justify right bottom)
+		)
+	)
+	(label "ICM_MOSI"
+		(at 77.47 105.41 180)
+		(effects
+			(font
+				(size 1.27 1.27)
+			)
+			(justify right bottom)
+		)
+	)
+	(label "ICM_MISO"
+		(at 77.47 107.95 180)
+		(effects
+			(font
+				(size 1.27 1.27)
+			)
+			(justify right bottom)
+		)
+	)
+	(label "BMI_SCLK"
+		(at 264.16 107.95 180)
+		(effects
+			(font
+				(size 1.27 1.27)
+			)
+			(justify right bottom)
+		)
+	)
+	(label "BMI_MOSI"
+		(at 264.16 110.49 180)
+		(effects
+			(font
+				(size 1.27 1.27)
+			)
+			(justify right bottom)
+		)
+	)
+	(label "BMI_ACC_SDO"
+		(at 264.16 113.03 180)
+		(effects
+			(font
+				(size 1.27 1.27)
+			)
+			(justify right bottom)
+		)
+	)
+	(label "BMI_GYR_SDO"
+		(at 264.16 115.57 180)
+		(effects
+			(font
+				(size 1.27 1.27)
+			)
+			(justify right bottom)
 		)
 	)
@@
 			)
 		)
+		(property "Description" "6-axis IMU, 4000dps/32g, SPI/I2C/I3C + AUX, LGA-14 2.5x3.0x0.81mm"
+			(at 110.49 110.49 0)
+			(hide yes)
+			(effects
+				(font
+					(size 1.27 1.27)
+				)
+			)
+		)
+		(property "Footprint_Status" "UNASSIGNED - land pattern not yet sourced from DS-000577"
+			(at 110.49 110.49 0)
+			(hide yes)
+			(effects
+				(font
+					(size 1.27 1.27)
+				)
+			)
+		)
+		(property "MPN" "ICM-45686"
+			(at 110.49 110.49 0)
+			(hide yes)
+			(effects
+				(font
+					(size 1.27 1.27)
+				)
+			)
+		)
+		(property "Manufacturer" "TDK InvenSense"
+			(at 110.49 110.49 0)
+			(hide yes)
+			(effects
+				(font
+					(size 1.27 1.27)
+				)
+			)
+		)
 		(instances
 			(project "imu-board"
@@
 			)
 		)
-		(property "Description" "6-axis IMU, 4000dps/32g, SPI/I2C/I3C + AUX, LGA-14 2.5x3.0x0.81mm"
-			(at 110.49 110.49 0)
-			(hide yes)
-			(effects
-				(font
-					(size 1.27 1.27)
-				)
-			)
-		)
-		(property "Footprint_Status" "UNASSIGNED - land pattern not yet sourced from DS-000577"
-			(at 110.49 110.49 0)
-			(hide yes)
-			(effects
-				(font
-					(size 1.27 1.27)
-				)
-			)
-		)
-		(property "MPN" "ICM-45686"
-			(at 110.49 110.49 0)
-			(hide yes)
-			(effects
-				(font
-					(size 1.27 1.27)
-				)
-			)
-		)
-		(property "Manufacturer" "TDK InvenSense"
-			(at 110.49 110.49 0)
-			(hide yes)
-			(effects
-				(font
-					(size 1.27 1.27)
-				)
-			)
-		))
+	)
 	(symbol
 		(lib_id "Sensor_Motion:BMI088")
@@
 			)
 		)
+		(property "Description" "6-axis IMU, separate accel + gyro dies, SPI/I2C, LGA-16 4.5x3mm"
+			(at 279.4 110.49 0)
+			(hide yes)
+			(effects
+				(font
+					(size 1.27 1.27)
+				)
+			)
+		)
+		(property "MPN" "BMI088"
+			(at 279.4 110.49 0)
+			(hide yes)
+			(effects
+				(font
+					(size 1.27 1.27)
+				)
+			)
+		)
+		(property "Manufacturer" "Bosch Sensortec"
+			(at 279.4 110.49 0)
+			(hide yes)
+			(effects
+				(font
+					(size 1.27 1.27)
+				)
+			)
+		)
 		(instances
 			(project "imu-board"
@@
 			)
 		)
-		(property "Description" "6-axis IMU, separate accel + gyro dies, SPI/I2C, LGA-16 4.5x3mm"
-			(at 279.4 110.49 0)
-			(hide yes)
-			(effects
-				(font
-					(size 1.27 1.27)
-				)
-			)
-		)
-		(property "MPN" "BMI088"
-			(at 279.4 110.49 0)
-			(hide yes)
-			(effects
-				(font
-					(size 1.27 1.27)
-				)
-			)
-		)
-		(property "Manufacturer" "Bosch Sensortec"
-			(at 279.4 110.49 0)
-			(hide yes)
-			(effects
-				(font
-					(size 1.27 1.27)
-				)
-			)
-		))
+	)
 	(symbol
 		(lib_id "Device:C")
