File: kicad/aeronode/aeronode.kicad_sch (KiCad schematic)
At the start: 1 part, among them U1 ConnectCore93

Commit message: [LIMA] kicad: add 474-pin ConnectCore93_LGA symbol; place it in aeronode
Generated deterministically from the HRM LGA pad tables (pp.43-82), 11 units:
POWER 29, GND 166, ENET1 14, ENET2 12, USB_SD 23, AUDIO 10, SERIAL 33,
DISPLAY 26, WIRELESS 9, GPIO_CTRL 27, NC 125 = 474.

Verified:
  - 474 pins read back, every pad number present, zero name mismatches vs HRM
  - symbol pin numbers == footprint pad names EXACTLY, both directions. This is
    the check that matters - a symbol and footprint that disagree each pass
    their own checks and produce a netlist that wires the wrong pads
  - all 11 units sit inside the A0 frame
  - ERC 526 violations, every one reconciled: 349 pin_not_connected (474 minus
    125 no-connect), 175 power_pin_not_driven (166 GND + 9 VSYS), 2
    pin_not_driven (SYS_RESET, ON_OFF). No structural errors

Near-miss worth recording: the first generation left one extra closing paren.
Nothing errored - list_symbols_in_library just returned count 0, and the
pre-existing ConnectCore93 symbol vanished from the listing too. A .kicad_sym
that fails to parse is indistinguishable from an empty one. Restored via git
checkout; generation now asserts paren balance and the read-back count.

aeronode.kicad_sch moves to A0 and carries all 11 units of U1 with the LGA
footprint attached. Schematic is placed, not yet wired.
Parts:
- removed U1: ConnectCore93, Digi:Digi_ConnectCore93_Castellated, symbol Digi:ConnectCore93
- added U1: ConnectCore93_LGA, symbol Digi:ConnectCore93_LGA

Commit message: [LIMA] aeronode: add J1 IMU connector, wired to LPSPI8 and LPSPI3
J1 (Conn_02x10_Odd_Even) carries the two IMUs on independent SPI buses, one per
chip, matching the split made on imu-board.

  ICM-45686 -> LPSPI8  SCK D17, SOUT E18, SIN E22, CS0 E19  (dedicated pads)
  BMI088    -> LPSPI3  SCK N29, SOUT M29, SIN R1, PCS0 P1   (UART7 pads)
  GPIO      -> BMI_GYR_CS C24, ICM_INT1 E28, ICM_INT2 E27,
               BMI_ACC_INT AA1, BMI_GYR_INT Y1

LPSPI4 and LPSPI5 were rejected - both land on SAI3's pads, which the A2B link
owns. LPSPI1 and LPSPI2 were rejected - both touch BOOT_MODE straps.

J1 pins 14 and 15 are deliberately the same net. The BMI088's two dies share
SCK and SDI but have separate SDO pins, so they cannot have independent buses;
imu-board brings both SDOs out separately and AeroNode ties them onto
LPSPI3_SIN, which is Bosch's topology with the chip selects arbitrating. The tie
lives on the host so it can be cut here if the dies ever need separate readback,
and so the ERC output-conflict does not have to be permanently excluded on the
sensor board.

Grounds interleaved between the SPI groups rather than bunched at one end, so a
ribbon or FFC has a return adjacent to each clock.

Verified: all 13 IMU nets land on exactly the intended endpoints (BMI_SDO on
three - two J1 pins plus R1); find_shorted_nets 0; ERC unconnected pins fell
349 -> 336, exactly the 13 module pins wired and nothing else disturbed.

+3V3 and GND on J1 are not yet tied to the module - the 3V3/1V8 outputs and the
166 GND pads belong to the power sheet. Until then +3V3 is legitimately a
single-pin net and ERC reports it as one.
Parts:
- added J1: IMU_BOARD, symbol Connector_Generic:Conn_02x10_Odd_Even
Connections:
- net ICM_SCLK: now reaches U1.D17 (SPI8_SCK)
- net ICM_SCLK: now also J1.3 (Pin_3)
- net ICM_MOSI: now reaches U1.E18 (SPI8_SOUT)
- net ICM_MOSI: now also J1.5 (Pin_5)
- net ICM_CS: now reaches U1.E19 (SPI8_CS0)
- net ICM_CS: now also J1.7 (Pin_7)
- net ICM_MISO: now reaches U1.E22 (SPI8_SIN)
- net ICM_MISO: now also J1.6 (Pin_6)
- net BMI_MOSI: now reaches U1.M29 (UART7_CTS)
- net BMI_MOSI: now also J1.13 (Pin_13)
- net BMI_SCLK: now reaches U1.N29 (UART7_RTS)
- net BMI_SCLK: now also J1.11 (Pin_11)
- net BMI_ACC_CS: now reaches U1.P1 (UART7_TX)
- net BMI_ACC_CS: now also J1.16 (Pin_16)
- net BMI_SDO: now reaches U1.R1 (UART7_RX)
- net BMI_SDO: now also J1.14 (Pin_14), J1.15 (Pin_15)
- net BMI_ACC_INT: now reaches U1.AA1 (GPIO2_IO06)
- net BMI_ACC_INT: now also J1.19 (Pin_19)
- net BMI_GYR_CS: now reaches U1.C24 (GPIO2_IO24)
- net BMI_GYR_CS: now also J1.17 (Pin_17)
- net ICM_INT2: now reaches U1.E27 (GPIO2_IO23)
- net ICM_INT2: now also J1.10 (Pin_10)
- net ICM_INT1: now reaches U1.E28 (GPIO2_IO22)
- net ICM_INT1: now also J1.9 (Pin_9)
- net BMI_GYR_INT: now reaches U1.Y1 (GPIO1_IO10)
- net BMI_GYR_INT: now also J1.20 (Pin_20)
- new net +3V3: J1.1 (Pin_1)
- new net GND: J1.12 (Pin_12), J1.18 (Pin_18), J1.2 (Pin_2), J1.4 (Pin_4), J1.8 (Pin_8)

Commit message: [LIMA] aeronode: power sheet stage 1 - module rails and all 166 GND pads
Sourced from HRM pp.13-15. Only three rails must be fed externally: VSYS
(3.7-6.0V), VSYS2 (2.7-6.0V) and NVCC_SD2 - the last is easy to miss, it is the
i.MX93 uSDHC2 IO supply and sits in the INPUT rail table.

  +5V         VSYS AL6/7/8 + VSYS2 AJ2/3/4, AK2/3/4   (9 pads, tied)
  +3V3        AK1, AL2, AL3, AM3, AM4                  (module output)
  +1V8        AH1, AH2, AH3, E5                        (module output)
  NVCC_SD2    F20 (MUX_3V3_1V8) + N1                   (LDO5 powers SD IO)
  SD_VSELECT  AH13 + AN5 (SD2_VSELECT)                 (Digi's recommendation)
  GND         all 166 pads

3V3_RF (F17/F18) deliberately NOT wired: it appears exactly once in 103 pages,
as a bare pad name, in neither the input nor output rail table. Direction
unknown, so it stays unconnected with the question written down.

Two symbol pin-type errors found and fixed. NVCC_SD2 was typed power_out when
it is an input - the generator classified by name pattern instead of by the
manual's own tables. And 3V3 on 5 pads / 1V8 on 4 pads are ONE internal rail
each, so typing every pad power_out raised 8 spurious output-to-output
conflicts; one driver kept per rail, duplicates set passive.

Near-miss: the first GND rail attempt connected nothing. I computed the pin
connection point as at+length, but in a .kicad_sym the 'at' IS the connection
point - the rails sat 2.54mm inside the pins. add_wire and batch_add_junction
both reported success. The only tell was the ERC count not moving: 336 stayed
336 when it should have hit 170. Now every bulk edit is checked against a
predicted ERC delta.

ERC 154: 148 pin_not_connected, 3 power_pin_not_driven (+5V/GND have no source
until stage 2), 3 pin_not_driven. All 8 pin_to_pin conflicts cleared.
Progression matched prediction at each step: 514 -> 170 -> 148.
Connections:
- net +3V3: now also U1.AK1 (3V3), U1.AL2 (3V3), U1.AL3 (3V3), U1.AM3 (3V3), U1.AM4 (3V3)
- net GND: now also U1.A25 (GND), U1.A4 (GND), U1.A5 (GND), U1.AF10 (GND), U1.AF11 (GND), U1.AF12 (GND), U1.AF13 (GND), U1.AF14 (GND), U1.AF15 (GND), U1.AF16 (GND), U1.AF17 (GND), U1.AF18 (GND), U1.AF19 (GND), U1.AF2 (GND), U1.AF20 (GND), U1.AF21 (GND), U1.AF22 (GND), U1.AF23 (GND), U1.AF24 (GND), U1.AF25 (GND), U1.AF26 (GND), U1.AF27 (GND), U1.AF28 (GND), U1.AF3 (GND), U1.AF4 (GND), U1.AF5 (GND), U1.AF6 (GND), U1.AF7 (GND), U1.AF8 (GND), U1.AF9 (GND), U1.AG16 (GND), U1.AG2 (GND), U1.AG23 (GND), U1.AG3 (GND), U1.AG4 (GND), U1.AG5 (GND), U1.AG6 (GND), U1.AG7 (GND), U1.AH14 (GND), U1.AH17 (GND), U1.AH19 (GND), U1.AH21 (GND), U1.AH4 (GND), U1.AH5 (GND), U1.AH8 (GND), U1.AJ1 (GND), U1.AJ14 (GND), U1.AJ17 (GND), U1.AJ20 (GND), U1.AJ26 (GND), U1.AJ5 (GND), U1.AJ6 (GND), U1.AJ7 (GND), U1.AJ9 (GND), U1.AK10 (GND), U1.AK11 (GND), U1.AK12 (GND), U1.AK13 (GND), U1.AK14 (GND), U1.AK17 (GND), U1.AK20 (GND), U1.AK23 (GND), U1.AK5 (GND), U1.AK6 (GND), U1.AK7 (GND), U1.AK8 (GND), U1.AK9 (GND), U1.AL10 (GND), U1.AL11 (GND), U1.AL14 (GND), U1.AL17 (GND), U1.AL4 (GND), U1.AL5 (GND), U1.AL9 (GND), U1.AM12 (GND), U1.AM15 (GND), U1.AM18 (GND), U1.AM20 (GND), U1.AM5 (GND), U1.AM6 (GND), U1.AN11 (GND), U1.AN14 (GND), U1.AN17 (GND), U1.AN20 (GND), U1.AN8 (GND), U1.B11 (GND), U1.B14 (GND), U1.B15 (GND), U1.B18 (GND), U1.B25 (GND), U1.B26 (GND), U1.B27 (GND), U1.B3 (GND), U1.B4 (GND), U1.B5 (GND), U1.B8 (GND), U1.C12 (GND), U1.C13 (GND), U1.C14 (GND), U1.C15 (GND), U1.C16 (GND), U1.C2 (GND), U1.C25 (GND), U1.C26 (GND), U1.C28 (GND), U1.C4 (GND), U1.C5 (GND), U1.D16 (GND), U1.D2 (GND), U1.D24 (GND), U1.D26 (GND), U1.D27 (GND), U1.D28 (GND), U1.D29 (GND), U1.D3 (GND), U1.D4 (GND), U1.E1 (GND), U1.E15 (GND), U1.E2 (GND), U1.E6 (GND), U1.E8 (GND), U1.F15 (GND), U1.F16 (GND), U1.F21 (GND), U1.F22 (GND), U1.G11 (GND), U1.G16 (GND), U1.G19 (GND), U1.G22 (GND), U1.G25 (GND), U1.G26 (GND), U1.G27 (GND), U1.G28 (GND), U1.G5 (GND), U1.G8 (GND), U1.H10 (GND), U1.H11 (GND), U1.H12 (GND), U1.H13 (GND), U1.H14 (GND), U1.H15 (GND), U1.H16 (GND), U1.H17 (GND), U1.H18 (GND), U1.H19 (GND), U1.H2 (GND), U1.H20 (GND), U1.H21 (GND), U1.H22 (GND), U1.H23 (GND), U1.H24 (GND), U1.H25 (GND), U1.H26 (GND), U1.H27 (GND), U1.H28 (GND), U1.H29 (GND), U1.H3 (GND), U1.H4 (GND), U1.H5 (GND), U1.H6 (GND), U1.H7 (GND), U1.H8 (GND), U1.H9 (GND), U1.M1 (GND), U1.T1 (GND), U1.Y29 (GND)
- net SD_VSELECT: now reaches U1.AN5 (SD2_VSELECT)
- net SD_VSELECT: now also U1.AH13 (SD_VSELECT)
- net +1V8: now reaches U1.AH1 (1V8)
- net +1V8: now also U1.AH2 (1V8), U1.AH3 (1V8), U1.E5 (1V8)
- net +5V: now reaches U1.AJ2 (VSYS2)
- net +5V: now also U1.AJ3 (VSYS2), U1.AJ4 (VSYS2), U1.AK2 (VSYS2), U1.AK3 (VSYS2), U1.AK4 (VSYS2), U1.AL6 (VSYS), U1.AL7 (VSYS), U1.AL8 (VSYS)
- net NVCC_SD2: now reaches U1.F20 (MUX_3V3_1V8)
- net NVCC_SD2: now also U1.N1 (NVCC_SD2)

Commit message: [LIMA] aeronode: power stage 2 - USB-C, PD sink, charger, battery; watchdog hazard found
Placed and wired J2 (USB-C), U2 (CYPD3177 PD sink), U3 (BQ25798 buck-boost
charger), J3 (2S LiFePO4 + BMS), R1 (/CE pull-up), R2 (PROG). Power path:
VBUS -> U2/U3, CC1/CC2, VBAT <-> J3, BAT_TS, REGN, CHG_CE_N, CHG_PROG,
VSYS_CHG.

HAZARD 1 REVISED, and it is worse than first stated. I had it as 'set VREG to
7.2V at boot before enabling charge'. The BQ25798 datasheet says:

  'when the REG_RST bit is set OR THE WATCHDOG TIMER EXPIRES, the registers are
   reset to default values with ICHG, VSYSMIN and VREG automatically returning
   to 1A, 7V and 8.4V'

VREG reverts to the Li-ion default on every watchdog expiry - 40/80/160s - with
no host involvement. A crash, hang, suspend or a paused driver silently applies
+1.2V of overcharge to a LiFePO4 pack. Setting the register once at boot is not
a fix, it is a fix that expires.

Three mitigations now required, all recorded in ARCHITECTURE.md:
  1. /CE pulled HIGH by R1 from REGN, so charging is off before any host boots.
     The datasheet is explicit the pin must never float.
  2. The I2C watchdog MUST be disabled after the host writes VREG=7.2V. This is
     a hardware-imposed FIRMWARE requirement and belongs in the driver bring-up
     notes, not left to be rediscovered.
  3. PROG resistor sets the 2S POR profile. Value still to be read from the
     datasheet's PROG table.

Still to do: VSYS_CHG->+5V buck (SYS sits at 7.0-7.3V for 2S, above the CC93's
6.0V absolute max, so it is not optional), VSYS overvoltage protection, the
VBUS_MIN/MAX and ISNK setpoint resistors, switching components, and I2C from
the CC93 to the charger for the VREG and watchdog writes.

ERC 209, no pin_to_pin conflicts. Cosmetic: J2's A4/B4 VBUS pins are stacked at
one coordinate so two identical VBUS labels sit on top of each other - one net,
redundant glyph, wants a click in eeschema.
Parts:
- added J2: USB-C PD / recovery, symbol Connector:USB_C_Receptacle_USB2.0_16P
- added J3: 2S LiFePO4 6Ah + BMS, symbol Connector_Generic:Conn_01x03
- added R1: 100k, symbol Device:R
- added R2: PROG 2S - TBD, symbol Device:R
- added U2: CYPD3177-24LQ, symbol Interface_USB:CYPD3177-24LQ
- added U3: BQ25798, symbol Battery_Management:BQ25798
Connections:
- net GND: now also J3.3 (Pin_3), R2.2, U2.19 (GND), U2.22 (GND), U2.25 (GND), U3.27 (GND)
- new net: J2.A1 (GND), J2.A12 (GND), J2.B1 (GND), J2.B12 (GND)
- new net BAT_TS: J3.2 (Pin_2), U3.16 (TS)
- new net CC1: J2.A5 (CC1), U2.15 (CC1)
- new net CC2: J2.B5 (CC2), U2.14 (CC2)
- new net CHG_CE_N: R1.2, U3.13 (~{CE})
- new net CHG_PROG: R2.1, U3.20 (PROG)
- new net REGN: R1.1, U3.5 (REGN)
- new net VBAT: J3.1 (Pin_1), U3.22 (BAT), U3.23 (BAT)
- new net VBUS: J2.A4 (VBUS), J2.A9 (VBUS), J2.B4 (VBUS), J2.B9 (VBUS), U2.18 (VBUS_IN), U3.2 (VBUS), U3.3 (VBUS)
- new net VSYS_CHG: U3.25 (SYS)

Commit message: [LIMA] aeronode: add 5V buck and PD setpoint dividers, all values sourced
U4 LMR33630ADDA converts the charger's SYS rail to +5V. Necessary, not
optional: SYS sits at ~7.0-7.3V for a 2S pack (VSYSMIN POR default 7V), above
the CC93's 6.0V absolute maximum.

  L1  4.7uH      7.3->5.0V at 3A, 400kHz, 30% ripple -> 4.4uH, standard 4.7uH
  R9/R10 100k/24.9k  V_FB = 1.000V from the datasheet, so Vout = 5.016V
  C1 10uF in, C2 47uF out, C3 100nF boot, C4 1uF VCC

5.016V leaves ~1V of headroom to the VSYS absolute maximum.

PD setpoints taken from the EZ-PD BCR datasheet Tables 2 and 3, not guessed.
These pins are resistor DIVIDERS from the chip's own VDDD 3.3V LDO, not single
pulldowns:

  VBUS_MIN    9V   5.1k / 1k     R3/R4
  VBUS_MAX    9V   5.1k / 1k     R5/R6
  ISNK_COARSE 3A   5.1k / 5.1k   R7/R8
  ISNK_FINE   0A   tied to GND

Min and max are deliberately identical - the datasheet's Note 3 says setting
them equal selects one specific voltage rather than accepting a range, so the
sink demands exactly 9V.

Recorded a trap from Note 2: the BCR does NOT enforce the ISNK current limit.
It is a request only, and the system must not exceed what the adapter offers -
the BQ25798's own input current limit has to do the enforcing. R7/R8 are not
protection.

Verified: every power-chain net endpoint count matched its prediction exactly
(SW_5V 3, BOOT_5V 2, VCC_BUCK 2, +5V 12, VSYS_CHG 4, FB_5V 3). ERC 200, down
from 204, with one isolated label left - PD_FAULT, which awaits a GPIO.
Parts:
- added C1: 10uF, symbol Device:C
- added C2: 47uF, symbol Device:C
- added C3: 100nF, symbol Device:C
- added C4: 1uF, symbol Device:C
- added L1: 4.7uH, symbol Device:L
- added R10: 24.9k, symbol Device:R
- added R3, R5, R7, R8: 5.1k, symbol Device:R
- added R4, R6: 1k, symbol Device:R
- added R9: 100k, symbol Device:R
- added U4: LMR33630ADDA, symbol Regulator_Switching:LMR33630ADDA
Connections:
- net +5V: now also C2.1, L1.2, R9.1
- net GND: now also U2.6 (ISNK_FINE), C1.2, C2.2, C4.2, R10.2, R4.2, R6.2, R8.2, U4.1 (GND), U4.9 (GND)
- net VSYS_CHG: now also C1.1, U4.2 (VIN), U4.3 (EN)
- net VBUS_MIN: now reaches U2.1 (VBUS_MIN)
- net VBUS_MIN: now also R3.2, R4.1
- net VBUS_MAX: now reaches U2.2 (VBUS_MAX)
- net VBUS_MAX: now also R5.2, R6.1
- net VDDD: now reaches U2.23 (VDDD)
- net VDDD: now also R3.1, R5.1, R7.1
- net ISNK_COARSE: now reaches U2.5 (ISNK_COARSE)
- net ISNK_COARSE: now also R7.2, R8.1
- net PD_FAULT: now reaches U2.9 (FAULT)
- new net BOOT_5V: C3.1, U4.7 (BOOT)
- new net FB_5V: R10.1, R9.2, U4.5 (FB)
- new net SW_5V: C3.2, L1.1, U4.8 (SW)
- new net VCC_BUCK: C4.1, U4.6 (VCC)

Commit message: [LIMA] aeronode: add charger I2C link and control GPIOs - the hazard mitigation path
This is the link the whole LiFePO4 mitigation depends on. Without it the host
cannot write VREG=7.2V, cannot disable the watchdog, and cannot enable charging.

  CHG_SCL    V1   I2C2_SCL     U3 pin 14   R11 10k pull-up
  CHG_SDA    W1   I2C2_SDA     U3 pin 15   R12 10k pull-up
  CHG_CE_N   AN4  GPIO2_IO18   U3 pin 13   host pulls LOW to enable
  CHG_INT_N  E3   GPIO2_IO19   U3 pin 21   R13 10k (open drain)
  PD_FAULT   P29  GPIO2_IO25   U2 pin 9
  PG_5V      R29  GPIO2_IO27   U4 pin 4    R14 100k (open drain)

10k on SCL/SDA is the BQ25798 datasheet's own figure, not a habit.

CHG_STAT_N drives D1 through R15 1k from +3V3, cathode to the charger's open
drain so it lights while charging. Pin polarity checked by reading D1's actual
pin coordinates rather than trusting the rotation - at rot 270 pin 1 is K and
pin 2 is A.

GPIO came from dropping CAN. Only AN4 and E3 were genuinely unallocated;
PD_FAULT and PG_5V use P29/R29, the CAN2 pads, free because CAN was dropped for
A2B. Recorded that reinstating CAN would take these two GPIOs back, and that
CAN1's T29/U29 are the next spare pair.

CHG_CE_N now has three connections - R1's pull-up disabling at POR, the charger,
and the GPIO that enables it. Mitigation 1 is complete: the charger is off until
software deliberately turns it on.

Also wrote the firmware obligations into ARCHITECTURE.md, since they are
hardware-imposed and invisible from the driver's side: set CELLS then VREG=7.20V,
disable the watchdog, and only then assert CE. Order matters - enabling charge
before setting VREG charges a LiFePO4 pack at the Li-ion voltage.

ERC 187, and zero isolated labels for the first time - every net reaches at
least two pins.
Parts:
- added D1: CHG, symbol Device:LED
- added R11, R12, R13: 10k, symbol Device:R
- added R14: 100k, symbol Device:R
- added R15: 1k, symbol Device:R
Connections:
- net +3V3: now also R11.1, R12.1, R13.1, R14.1, R15.1
- net CHG_CE_N: now also U1.AN4 (GPIO2_IO18)
- net PD_FAULT: now also U1.P29 (CAN2_TX)
- net PG_5V: now reaches U1.R29 (CAN2_RX)
- net PG_5V: now also U4.4 (PG), R14.2
- net CHG_SCL: now reaches U1.V1 (I2C2_SCL)
- net CHG_SCL: now also U3.14 (SCL), R11.2
- net CHG_SDA: now reaches U1.W1 (I2C2_SDA)
- net CHG_SDA: now also U3.15 (SDA), R12.2
- net CHG_STAT_N: now reaches U3.1 (STAT)
- net CHG_STAT_N: now also D1.1 (K)
- net CHG_INT_N: now reaches U3.21 (~{INT})
- net CHG_INT_N: now also U1.E3 (GPIO2_IO19), R13.2
- new net CHG_LED_A: D1.2 (A), R15.2

Commit message: [LIMA] aeronode: add VSYS overvoltage protection (U5 LTC4364 surge stopper)
VSYS has a 6.0V absolute maximum, the buck outputs 5.016V, and VSYS_CHG sits at
7.0-7.3V behind it. Two realistic faults put that on the module: the buck's
high-side FET failing short, or - the classic - the feedback lower leg going
open, which makes FB read 0V and drives the buck to full duty.

A TVS cannot do this job: a 5V TVS clamps near 9V, far past the limit. Nor can
a Zener-referenced discrete - the usable window is 5.12V to 6.0V and +/-5%
Zener tolerance either nuisance-trips or misses. It needs a precision reference.

U5 LTC4364 inserted between buck and module. The buck output becomes +5V_RAW;
+5V stays the protected rail into VSYS, so no module-side rework.

  R16/R17  34k/10k    OV  trip 5.500V
  R18/R19  22.1k/10k  UV  trip 4.013V
  R20/R21  30.1k/10k  FB  clamp 5.013V
  R22      15m        sense, 50mV/3A
  C5       0.22uF     TMR

All from the datasheet's 1.25V reference; every divider lands on an E96 1%
value almost exactly. OVP_FLT_N goes to pad T29.

Note the feedback divider R9/R10 deliberately senses +5V_RAW, not the protected
side. Sensing downstream would mean that if the OVP ever opened, the buck would
lose feedback and drive to full duty - the protection would cause the fault it
exists to prevent.

Four open items recorded in ARCHITECTURE.md and NOT to be skipped before fab:
Q1 is unspecified and must be chosen on SOA (it dissipates (7.3-5.0)xI during a
clamped surge); DGATE is left open on the assumption a single-source design does
not need the ideal-diode FET, which is unconfirmed; the LTC4364 is designed for
12-80V rails and is being used near its 4V floor, so a purpose-built low-voltage
OVP part would be better if someone authors the symbol; ENOUT unused.

Verified: all nine OVP nets match their predicted endpoint counts, no isolated
labels, no pin_to_pin conflicts. ERC 189.
Parts:
- added C5: 0.22uF, symbol Device:C
- added Q1: NMOS pass - TBD, symbol Device:Q_NMOS
- added R16: 34k, symbol Device:R
- added R17, R19, R21: 10k, symbol Device:R
- added R18: 22.1k, symbol Device:R
- added R20: 30.1k, symbol Device:R
- added R22: 15m, symbol Device:R
- added U5: LTC4364CMS, symbol Power_Management:LTC4364CMS
Connections:
- net +5V: now also R20.1, R22.2, U5.1 (OUT); no longer C2.1, L1.2, R9.1
- net GND: now also C5.2, R17.2, R19.2, R21.2, U5.12 (GND)
- net OVP_FLT_N: now reaches U1.T29 (CAN1_TX)
- net OVP_FLT_N: now also U5.13 (~{FLT})
- new net +5V_RAW: C2.1, L1.2, Q1.D, R16.1, R18.1, R9.1, U5.8 (VCC), U5.9 (~{SHDN})
- new net OVP_FB: R20.2, R21.1, U5.16 (FB)
- new net OVP_HGATE: Q1.G, U5.6 (HGATE)
- new net OVP_OV: R16.2, R17.1, U5.11 (OV)
- new net OVP_SENSE: Q1.S, R22.1, U5.2 (SENSE), U5.5 (SOURCE)
- new net OVP_TMR: C5.1, U5.15 (TMR)
- new net OVP_UV: R18.2, R19.1, U5.10 (UV)
