File: kicad/aeronode/aeronode.kicad_sch (KiCad schematic)
At the start: 73 parts, among them J1 IMU_BOARD, J2 USB-C PD / recovery, J3 2S LiFePO4 6Ah + BMS, Q1 NMOS pass - TBD, SW1 ON/OFF, U1 ConnectCore93_LGA, U10 BMP390, U2 CYPD3177-24LQ, U3 BQ25798, U4 LMR33630ADDA, U5 LTC4364CMS, U6 BME690, U7 DAN-F10N, U9 MMC5983MA

Commit message: [LIMA] aeronode: assign 66/73 footprints, set 4-layer stackup; RETRACT the 8-layer claim
CORRECTION first. I previously said this board needed 8+ layers with via-in-pad
because it carries a 474-pad LGA at 1.27mm pitch. That was wrong, and wrong for
a bad reason: I judged it from the pad count without counting the escape load.

  GND                      166  via straight to plane, no routing
  NC / RESERVED            125  nothing to connect
  power                     18  via to plane
  signal pads left unused  128  not connected
  SIGNALS ACTUALLY WIRED    37  the only real escape

37 of 474 pads is 8%, and 1.27mm pitch is generous by BGA standards. Ordinary
dogbone vias at 4/4 mil will do it. 4 layers is sufficient, as Peter asked.

Stackup set: F.Cu signal, In1.Cu ground plane, In2.Cu power plane, B.Cu signal.
The 166 GND pads are what makes it easy - each is one via to In1, which also
gives the switching converters a solid return directly beneath them.

Footprints: 66 of 73 assigned. 0402 for R and small C, 0603 for 1-10uF and the
LEDs, 0805 for the 47uF bulk, 1206 for the R22 current sense. Inductors SRN6028
and SRN4018. Note U2-U5 needed explicit assignment - the stock symbols carry
default footprints but those do not copy to the instance on placement.

THREE LEFT DELIBERATELY EMPTY rather than given a wrong land pattern:
  U7  DAN-F10N    author from scratch, 56 pads, 20x20mm, nothing comparable
  U9  MMC5983MA   generic LGA-16 3x3 exists but must be verified vs MEMSIC's
  U10 BMP390      no Bosch LGA-10 2x2; ST's HLGA-10 fits the envelope but is
                  a different vendor's land pattern

TWO ASSIGNED BUT PROVISIONAL: Q1's SOT-23 is a placeholder package only, the
OVP FET still needs selecting on SOA; L1/L2 packages suit the inductance but
saturation current has not been checked against 3A plus ripple.

Also worth recording: my first two footprint audits gave wrong counts because
the regex matched neighbouring components' properties. The numbers he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
Parts:
- C1, C10, C11, C12, C15, C18, C4, C8, C9: footprint (none) -> Capacitor_SMD:C_0603_1608Metric
- C13, C14, C16, C17, C19, C20, C21, C22, C3, C5, C6, C7: footprint (none) -> Capacitor_SMD:C_0402_1005Metric
- C2: footprint (none) -> Capacitor_SMD:C_0805_2012Metric
- D1, D2, D3, D4: footprint (none) -> LED_SMD:LED_0603_1608Metric
- J1: footprint (none) -> Connector_PinHeader_2.54mm:PinHeader_2x10_P2.54mm_Vertical
- J2: footprint (none) -> Connector_USB:USB_C_Receptacle_HCTL_HC-TYPE-C-16P-01A
- J3: footprint (none) -> Connector_PinHeader_2.54mm:PinHeader_1x03_P2.54mm_Vertical
- L1: footprint (none) -> Inductor_SMD:L_Bourns-SRN6028
- L2: footprint (none) -> Inductor_SMD:L_Bourns-SRN4018
- Q1: footprint (none) -> Package_TO_SOT_SMD:SOT-23
- R1, R10, R11, R12, R13, R14, R15, R16, R17, R18, R19, R2, R20, R21, R23, R24, R25, R26, R27, R28, R29, R3, R30, R31, R4, R5, R6, R7, R8, R9: footprint (none) -> Resistor_SMD:R_0402_1005Metric
- R22: footprint (none) -> Resistor_SMD:R_1206_3216Metric
- SW1: footprint (none) -> Button_Switch_SMD:SW_Push_1P1T_NO_CK_KMR2
- U1: footprint (none) -> Digi:Digi_ConnectCore93_LGA
- U2: footprint (none) -> Package_DFN_QFN:QFN-24-1EP_4x4mm_P0.5mm_EP2.75x2.75mm
- U3: footprint (none) -> Package_DFN_QFN:Texas_RQM0029A_VQFN-29_4x4mm_P0.4mm
- U4: footprint (none) -> Package_SO:Texas_HSOP-8-1EP_3.9x4.9mm_P1.27mm_ThermalVias
- U5: footprint (none) -> Package_SO:MSOP-16_3x4.039mm_P0.5mm
