File: kicad/aeronode/aeronode.kicad_sch (KiCad schematic)
At the start: 73 parts, among them J1 IMU_BOARD, J2 USB-C PD / recovery, J3 2S LiFePO4 6Ah + BMS, Q1 NMOS pass - TBD, SW1 ON/OFF, U1 ConnectCore93_LGA, U10 BMP390, U2 CYPD3177-24LQ, U3 BQ25798, U4 LMR33630ADDA, U5 LTC4364CMS, U6 BME690, U7 DAN-F10N, U9 MMC5983MA

Commit message: [LIMA] kicad: author DAN-F10N footprint from u-blox Integration Manual Fig 18
100 pads: 56 numbered edge pads (1.50x0.80 on 1.10 pitch, rows at +/-8.95) plus a
44-pad unnumbered ground array (1.10 sq on a 1.90 grid) assigned to pad 1 (GND).

Geometry recovered from the bitmap figure by connected-component analysis and
reconciled against Table 27. Two traps recorded in ARCHITECTURE.md and lib/README.md:

- Blob sizes fitted 130 px/mm self-consistently and were wrong; pitches fitted 127.3.
  Anti-aliasing inflates sizes but not centroids, so calibrate on distances.
- Datasheet Fig 3 and Integration Manual Fig 18 disagree on pin-1 orientation by 90 deg;
  the 4-fold symmetric ground array hides the conflict. Built to Fig 3 (pin 1 top-left).

Verified: 56/56 pins match the symbol, 0 overlaps, min copper gap 0.300 mm, paste
margin confirmed live via pcbnew. Assigned to U7; footprints now 81 of 83.

Co-Authored-By: Claude Opus 5 <noreply@anthropic.com>
Parts:
- U7: footprint (none) -> ublox:ublox_DAN-F10N
Changed lines of the file:
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@@
 			)
 		)
-		(property "Footprint" ""
+		(property "Footprint" "ublox:ublox_DAN-F10N"
 			(at 1060.45 720.09 0)
 			(hide yes)
