File: kicad/aeronode/aeronode.kicad_pcb (KiCad board)
At the start: 2 copper layers, 0 parts

Commit message: [LIMA] aeronode: assign 66/73 footprints, set 4-layer stackup; RETRACT the 8-layer claim
CORRECTION first. I previously said this board needed 8+ layers with via-in-pad
because it carries a 474-pad LGA at 1.27mm pitch. That was wrong, and wrong for
a bad reason: I judged it from the pad count without counting the escape load.

  GND                      166  via straight to plane, no routing
  NC / RESERVED            125  nothing to connect
  power                     18  via to plane
  signal pads left unused  128  not connected
  SIGNALS ACTUALLY WIRED    37  the only real escape

37 of 474 pads is 8%, and 1.27mm pitch is generous by BGA standards. Ordinary
dogbone vias at 4/4 mil will do it. 4 layers is sufficient, as Peter asked.

Stackup set: F.Cu signal, In1.Cu ground plane, In2.Cu power plane, B.Cu signal.
The 166 GND pads are what makes it easy - each is one via to In1, which also
gives the switching converters a solid return directly beneath them.

Footprints: 66 of 73 assigned. 0402 for R and small C, 0603 for 1-10uF and the
LEDs, 0805 for the 47uF bulk, 1206 for the R22 current sense. Inductors SRN6028
and SRN4018. Note U2-U5 needed explicit assignment - the stock symbols carry
default footprints but those do not copy to the instance on placement.

THREE LEFT DELIBERATELY EMPTY rather than given a wrong land pattern:
  U7  DAN-F10N    author from scratch, 56 pads, 20x20mm, nothing comparable
  U9  MMC5983MA   generic LGA-16 3x3 exists but must be verified vs MEMSIC's
  U10 BMP390      no Bosch LGA-10 2x2; ST's HLGA-10 fits the envelope but is
                  a different vendor's land pattern

TWO ASSIGNED BUT PROVISIONAL: Q1's SOT-23 is a placeholder package only, the
OVP FET still needs selecting on SOA; L1/L2 packages suit the inductance but
saturation current has not been checked against 3A plus ripple.

Also worth recording: my first two footprint audits gave wrong counts because
the regex matched neighbouring components' properties. The numbers he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
Other:
- copper layers 2 -> 4
Changed lines of the file:
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@@
 		(48 "B.Fab" user)
 		(49 "F.Fab" user)
+		(1 "In1.Cu" power)
+		(2 "In2.Cu" power)
 	)
 	(setup
