File: kicad/aeronode/aeronode.kicad_pcb (KiCad board)
At the start: 4 copper layers, 0 parts

Commit message: [LIMA] kicad: import netlist to PCB, draw 90x70 outline, fix unconnectable Q1
Netlist import: 73 footprints, 385 nets. kicad-cli has no update-pcb-from-schematic
and KiCad 10's pcbnew SWIG exposes no BOARD_NETLIST_UPDATER, so this is a scripted
import verified by re-reading the saved board: 806 nodes checked, 0 mismatches, and
kicad-cli pcb drc reports schematic_parity 0.

Q1 could never have worked. It used Device:Q_NMOS, whose pin NUMBERS are the letters
D/G/S, against a SOT-23 footprint with pads 1/2/3 - all three pads bound to nothing,
so the OVP pass FET was electrically absent. ERC cannot see this; it only exists at
the symbol/footprint boundary. KiCad 10 ships no Q_NMOS_* numbered variants, so
authored AeroNode:NMOS_GSD (Q_NMOS graphics, pins 1=G/2=S/3=D). Not patched into the
schematic's cached lib_symbols, which Update-Symbols-from-Library would revert.

Outline 90x70mm, R3 corners, 4x M3 NPTH on an 80x60 pattern. Size is an ASSUMPTION -
3010mm2 of courtyard over 73 parts gives ~48% density. Cheap to change now, not later.
Anchors placed: CC93, GNSS top-right (sky view, away from switchers), IMU header on
the right edge, USB-C flush with the bottom edge, battery bottom-centre.

Two placement errors caught by measurement, not inspection: J1 rotated 90deg landed
18.7mm off the board (its native courtyard is already tall), and J3 hung 0.89mm past
the edge because a pin header's origin is pin 1, not the courtyard centre. Placement
now targets courtyard centres.

DRC 0 violations. Fixed U10's 0.7mm silk text. Accepted one residual via a rule scoped
to J2 only: the USB-C receptacle's own GND holes sit 0.1847mm from its own NPTH holes,
fixed by the connector's mechanics. Fab must confirm 0.18mm hole-to-hole.

Also corrected the record: 73 components, not 83 - the old number counted symbol units
and U1 is an 11-unit symbol.

Co-Authored-By: Claude Opus 5 <noreply@anthropic.com>
Parts:
- added C1: 10uF, C_0603_1608Metric, F.Cu at (156.5, 45.8)
- added C10: 10uF, C_0603_1608Metric, F.Cu at (206.5, 45.8)
- added C11: 10uF, C_0603_1608Metric, F.Cu at (212.5, 45.8)
- added C12: 10uF, C_0603_1608Metric, F.Cu at (218.5, 45.8)
- added C13: 100nF, C_0402_1005Metric, F.Cu at (223.9, 45.5)
- added C14: 100nF, C_0402_1005Metric, F.Cu at (228.8, 45.5)
- added C15: 10uF, C_0603_1608Metric, F.Cu at (234.2, 45.8)
- added C16: 100nF, C_0402_1005Metric, F.Cu at (239.7, 45.5)
- added C17: 100nF, C_0402_1005Metric, F.Cu at (244.6, 45.5)
- added C18: 10uF, C_0603_1608Metric, F.Cu at (250.0, 45.8)
- added C19: 100nF, C_0402_1005Metric, F.Cu at (255.4, 45.5)
- added C2: 47uF, C_0805_2012Metric, F.Cu at (162.7, 46.0)
- added C20: 100nF, C_0402_1005Metric, F.Cu at (260.3, 45.5)
- added C21: 100nF, C_0402_1005Metric, F.Cu at (265.2, 45.5)
- added C22: 100nF, C_0402_1005Metric, F.Cu at (270.0, 45.5)
- added C3: 100nF, C_0402_1005Metric, F.Cu at (168.4, 45.5)
- added C4: 1uF, C_0603_1608Metric, F.Cu at (173.8, 45.8)
- added C5: 0.22uF, C_0402_1005Metric, F.Cu at (179.3, 45.5)
- added C6: 47nF, C_0402_1005Metric, F.Cu at (184.1, 45.5)
- added C7: 47nF, C_0402_1005Metric, F.Cu at (189.0, 45.5)
- added C8: 4.7uF, C_0603_1608Metric, F.Cu at (194.5, 45.8)
- added C9: 10uF, C_0603_1608Metric, F.Cu at (200.5, 45.8)
- added D1: CHG, LED_0603_1608Metric, F.Cu at (275.5, 45.8)
- added D2: RED, LED_0603_1608Metric, F.Cu at (281.6, 45.8)
- added D3: GREEN, LED_0603_1608Metric, F.Cu at (156.5, 50.8)
- added D4: BLUE, LED_0603_1608Metric, F.Cu at (162.6, 50.8)
- added H1: M3 NPTH, MountingHole_3.2mm_M3, F.Cu at (25.0, 25.0)
- added H2: M3 NPTH, MountingHole_3.2mm_M3, F.Cu at (105.0, 25.0)
- added H3: M3 NPTH, MountingHole_3.2mm_M3, F.Cu at (25.0, 85.0)
- added H4: M3 NPTH, MountingHole_3.2mm_M3, F.Cu at (105.0, 85.0)
- added J1: IMU_BOARD, PinHeader_2x10_P2.54mm_Vertical, F.Cu at (102.7, 54.6)
- added J2: USB-C PD / recovery, USB_C_Receptacle_HCTL_HC-TYPE-C-16P-01A, F.Cu at (40.0, 85.8)
- added J3: 2S LiFePO4 6Ah + BMS, PinHeader_1x03_P2.54mm_Vertical, F.Cu at (60.0, 81.0)
- added L1: 4.7uH, L_Bourns-SRN6028, F.Cu at (200.0, 53.3)
- added L2: 1.0uH, L_Bourns-SRN4018, F.Cu at (209.0, 52.3)
- added Q1: NMOS pass - TBD, SOT-23, F.Cu at (216.5, 51.7)
- added R1: 100k, R_0402_1005Metric, F.Cu at (222.4, 50.5)
- added R10: 24.9k, R_0402_1005Metric, F.Cu at (266.6, 50.5)
- added R11: 10k, R_0402_1005Metric, F.Cu at (271.5, 50.5)
- added R12: 10k, R_0402_1005Metric, F.Cu at (276.4, 50.5)
- added R13: 10k, R_0402_1005Metric, F.Cu at (281.3, 50.5)
- added R14: 100k, R_0402_1005Metric, F.Cu at (156.0, 80.0)
- added R15: 1k, R_0402_1005Metric, F.Cu at (160.9, 80.0)
- added R16: 34k, R_0402_1005Metric, F.Cu at (165.8, 80.0)
- added R17: 10k, R_0402_1005Metric, F.Cu at (170.7, 80.0)
- added R18: 22.1k, R_0402_1005Metric, F.Cu at (175.6, 80.0)
- added R19: 10k, R_0402_1005Metric, F.Cu at (180.5, 80.0)
- added R2: 6.04k, R_0402_1005Metric, F.Cu at (227.3, 50.5)
- added R20: 30.1k, R_0402_1005Metric, F.Cu at (185.4, 80.0)
- added R21: 10k, R_0402_1005Metric, F.Cu at (190.3, 80.0)
- added R22: 15m, R_1206_3216Metric, F.Cu at (196.6, 80.6)
- added R23: 5.24k, R_0402_1005Metric, F.Cu at (202.8, 80.0)
- added R24: 30.31k, R_0402_1005Metric, F.Cu at (207.8, 80.0)
- added R25: 4.7k, R_0402_1005Metric, F.Cu at (212.7, 80.0)
- added R26: 4.7k, R_0402_1005Metric, F.Cu at (217.6, 80.0)
- added R27: 100R, R_0402_1005Metric, F.Cu at (222.5, 80.0)
- added R28: 160R, R_0402_1005Metric, F.Cu at (227.4, 80.0)
- added R29: 150R, R_0402_1005Metric, F.Cu at (232.3, 80.0)
- added R3: 5.1k, R_0402_1005Metric, F.Cu at (232.2, 50.5)
- added R30: 68R, R_0402_1005Metric, F.Cu at (237.2, 80.0)
- added R31: 10k, R_0402_1005Metric, F.Cu at (242.1, 80.0)
- added R4: 1k, R_0402_1005Metric, F.Cu at (237.1, 50.5)
- added R5: 5.1k, R_0402_1005Metric, F.Cu at (242.1, 50.5)
- added R6: 1k, R_0402_1005Metric, F.Cu at (247.0, 50.5)
- added R7: 5.1k, R_0402_1005Metric, F.Cu at (251.9, 50.5)
- added R8: 5.1k, R_0402_1005Metric, F.Cu at (256.8, 50.5)
- added R9: 100k, R_0402_1005Metric, F.Cu at (261.7, 50.5)
- added SW1: ON/OFF, SW_Push_1P1T_NO_CK_KMR2, F.Cu at (248.9, 81.3)
- added U1: ConnectCore93_LGA, Digi_ConnectCore93_LGA, F.Cu at (52.0, 51.0)
- added U10: BMP390, Bosch_BMP390_LGA-10_2x2mm, F.Cu at (187.9, 148.2)
- added U2: CYPD3177-24LQ, QFN-24-1EP_4x4mm_P0.5mm_EP2.75x2.75mm, F.Cu at (238.6, 88.8)
- added U3: BQ25798, Texas_RQM0029A_VQFN-29_4x4mm_P0.4mm, F.Cu at (247.1, 88.6)
- added U4: LMR33630ADDA, Texas_HSOP-8-1EP_3.9x4.9mm_P1.27mm_ThermalVias, F.Cu at (256.6, 88.9)
- added U5: LTC4364CMS, MSOP-16_3x4.039mm_P0.5mm, F.Cu at (266.7, 88.4)
- added U6: BME690, Bosch_LGA-8_3x3mm_P0.8mm_ClockwisePinNumbering, F.Cu at (274.8, 88.1)
- added U7: DAN-F10N, ublox_DAN-F10N, F.Cu at (91.5, 41.0)
- added U9: MMC5983MA, LGA-16_3x3mm_P0.5mm, F.Cu at (181.6, 148.7)
Other:
- board outline added: 90 x 70 mm

Commit message: [LIMA] kicad: place all 73 parts, strip stray DVK keepouts from CC93 footprint
Placement complete: DRC 0 violations, schematic parity 0, 466 unconnected
(nothing routed). Board 90x70 confirmed; U9 stays on this board.

Removed 6 rule-area keepout zones from Digi_ConnectCore93_LGA that came in with
the Altium DVK library. Each spanned all 32 copper layers with tracks/vias/pads/
copperpour disallowed, sitting +/-37mm from the module centre - the dev kit's
mounting-hole keepouts, not the module's. They were invisible until a buck
inductor pad landed in one. Left in, they would have silently blocked routing
over large areas. 474 pads verified unchanged.

Placement took two passes because the first was electrically wrong. Zone packing
largest-first was DRC-clean but left U4's input caps 13-18mm and U3's up to 21mm
from their ICs - a 20mm high-di/dt loop is an EMI defect. Pass 2 re-placed every
passive at the nearest free spot to the centroid of the owner IC's pads it shares
a net with, excluding GND so decoupling targets the supply pin. U4 caps now
4.1-5.0mm, U3 caps 3.4-5.0mm - against the package edge.

Silk: 118 auto-placement silk violations resolved by moving passive/IC refs to
F.Fab. Silk keeps J1-J3, SW1, H1-H4 and polarity/pin-1 marks.

Known gaps recorded: passive rotations not optimised (all at 0deg), loop AREAS
not yet minimised, GNSS-to-buck 29.4mm is the tightest coupling margin.

Co-Authored-By: Claude Opus 5 <noreply@anthropic.com>
Parts:
- moved D2 259.0 mm to (23.1, 29.9)
- moved U6 251.7 mm to (31.8, 22.4)
- moved D1 235.5 mm to (41.7, 73.9)
- moved C22 230.7 mm to (40.3, 24.1)
- moved SW1 230.6 mm to (23.4, 32.8)
- moved R8 229.4 mm to (29.0, 78.3)
- moved R12 228.7 mm to (49.7, 80.7)
- moved R13 227.4 mm to (55.6, 77.5)
- moved C21 224.4 mm to (42.0, 21.7)
- moved C20 224.0 mm to (37.1, 27.0)
- moved R7 222.0 mm to (31.6, 78.1)
- moved C19 221.8 mm to (34.4, 26.8)
- moved R11 221.1 mm to (52.3, 79.6)
- moved C17 220.9 mm to (23.8, 35.6)
- moved R6 220.5 mm to (28.0, 76.8)
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