File: kicad/audio-board/audio-board.kicad_sch (KiCad schematic)
At the start: 45 parts, among them J1 TO_CM5, J2 VBAT_IN, U1 ADAU1861, U10 ADP7118AUJZ-3.3-R7, U2 ADXL354CEZ, U3 LTC6242, U4 IM72D128VV01, U5 AD2428WBCPZ, U6 SN74LVC8T245PWR, U7 SN74LVC8T245PWR, U8 PCA9517ADP, U9 ADP7118AUJZ-1.8-R7

Commit message: [LIMA] cross U5's DTX0/DRX0 to RP1 as a second I2S/TDM lane, per Peter
U5 DTX0 -> U6's freed A4/B4 (up, DIR=1V8) -> J1 pin 10 (DTX0_3V3). U5 DRX0 <- U7's freed A2/B2
(down, DIR=AGND) <- J1 pin 11 (DRX0_3V3). Both reuse the exact channels SPT1's old host path
vacated last pass - no new translator hardware. This lane rides the SAME BCLK_3V3/FSYNC_3V3 that
SPT0 already uses; RP1 would need a second SAI/I2S peripheral slaved to that one shared clock pair,
mirroring the pattern this board already uses locally for SPT0/SPT1. J1 grew from 9 to 11 pins to
carry the two new signals (pin 4 stays spare from the earlier SPT1 reroute).

Caught and fixed before committing: my first draft of the note claimed "DTX0/DTX1 both now wired"
implying both reach RP1 - wrong. DTX1 goes to U1 (SPT1's local link), not to the host. Corrected
the channel arithmetic accordingly: the decision record's "two lanes x two slots = four channels"
figure assumed DTX0 AND DTX1 both reaching RP1; that's no longer the design. RP1's actual upstream
A2B capacity via U5 is now one lane (DTX0), up to 2 slots - a real reduction flagged as a fresh
open item, not the same question the decision record sized.

Also flagged, not asserted as solved: whether RP1's driver stack can actually run a second I2S
peripheral against an externally-shared, already-used BCLK/FSYNC pair is asserted by this
schematic's topology, not measured. And mic3's data (now landing at U5 via DRX1) can only reach
RP1 by competing with upstream A2B traffic for DTX0's 2 slots - worth confirming on the bench.

ERC clean, no shorts, no overlaps.
Parts:
- removed J1: TO_CM5, symbol Connector_Generic:Conn_01x09
- added J1: TO_CM5, symbol Connector_Generic:Conn_01x11
Connections:
- net 3V3_CM5: now also J1.8 (Pin_8)
- net AGND: now also J1.9 (Pin_9)
- net BCLK_3V3: now also J1.1 (Pin_1)
- net FSYNC_3V3: now also J1.2 (Pin_2)
- net SCL_3V3: now also J1.6 (Pin_6)
- net SDATAI_0_3V3: now also J1.5 (Pin_5)
- net SDATAO_0_3V3: now also J1.3 (Pin_3)
- net SDA_3V3: now also J1.7 (Pin_7)
- net DTX0_3V3: now reaches U6.18 (B4)
- net DTX0_3V3: now also J1.10 (Pin_10)
- net DTX0: now reaches U6.6 (A4)
- net DTX0: now also U5.12 (DTX0/IO3)
- net DRX0: now reaches U5.14 (DRX0/IO5)
- net DRX0: now also U7.4 (A2)
- net DRX0_3V3: now reaches U7.20 (B2)
- net DRX0_3V3: now also J1.11 (Pin_11)
Other:
- note added: "I2S + I2C crossing to the host (CM5/RP1), per docs/audio-board-level-shifter.md (this note's "1860" is the same silicon as our 1861, UG-2257 p.1) and Decision D in docs/audio-board-decision-record.md. SIX signals now cross to the host, on TWO I2S/TDM lanes sharing ONE clock pair: BCLK_0, FSYNC_0, SDATAO_0, and NOW U5's DTX0 go UP through U6 (SN74LVC8T245, DIR=1V8 so A->B, using the two channels f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"
- note removed: "I2S + I2C crossing to the host (CM5/RP1), per docs/audio-board-level-shifter.md (this note's "1860" is the same silicon as our 1861, UG-2257 p.1) and Decision D in docs/audio-board-decision-record.md. FOUR signals cross to the host now (was five - see SPT1 below): BCLK_0, FSYNC_0, SDATAO_0 go UP through U6 (SN74LVC8T245, DIR=1V8 so A->B); SDATAI_0 (host playback) goes DOWN through U7 (same part, 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"

Commit message: [LIMA] retire 3V3_CM5 - merge into 3V3_ACCEL, per Peter: only VBAT crosses the board boundary
Peter corrected an assumption I'd been carrying since the level-shifter work: there is no 3.3V
rail arriving from the CM5/aeronode side at all, only VBAT. The "3V3_CM5" net I'd invented as
"assumed supplied by the CM5 header" never had a real source - U10 (the local 3.3V LDO, already
feeding the accelerometer as 3V3_ACCEL) is the only 3.3V this board actually has.

Merged 3V3_CM5 into 3V3_ACCEL everywhere it appeared: U6/U7's VCCB, U8's VCC(B) and EN, and
R6/R7's pull-up reference. Removed the now-wrong 3V3_CM5 PWR_FLAG (there was never a real board-
boundary supply to flag) and its J1 pin - J1 pins 4 and 8 are both spare now. RP1 keeps its own
3.3V supply on its own board, as it already must; the two boards interoperate on a shared ground
and translated signal lines, same as any two independently-supplied boards.

Sharpened, not silently absorbed: U10 (ADP7118, 200mA/rail) now carries the accelerometer's own
load plus both I2S translators' VCCB plus the I2C repeater plus two 4.7k pull-ups. Still almost
certainly fine, but it's a real aggregate now, not just "the accelerometer's load" - flagged in
the power note as worth computing before layout.

ERC clean, no shorts, no overlaps.
Connections:
- net 3V3_ACCEL: now also R6.1, R7.1, U6.23 (VCCB), U6.24 (VCCB), U7.23 (VCCB), U7.24 (VCCB), U8.5 (EN), U8.8 (VCC(B))
- removed net 3V3_CM5: J1.8 (Pin_8), R6.1, R7.1, U6.23 (VCCB), U6.24 (VCCB), U7.23 (VCCB), U7.24 (VCCB), U8.5 (EN), U8.8 (VCC(B))
Other:
- note added: "Power in: VBAT from the aeronode board (U9/U10, J2). This is the ONLY supply arriving on this board - Peter confirmed no 3.3V rail comes over from the CM5 side at all. VBAT is aeronode's raw 2S LiFePO4 pack net (ahead of its charger/buck stage) - per kicad/aeronode/doc/ARCHITECTURE.md: "the pack never falls below 5.0V" and "the pack sits at 7.2V" at full charge, so VBAT runs 5.0-7.3V. Fetched fro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"
- note removed: "Power in: VBAT from the aeronode board (U9/U10, J2). VBAT is aeronode's raw 2S LiFePO4 pack net (ahead of its charger/buck stage) - per kicad/aeronode/doc/ARCHITECTURE.md: "the pack never falls below 5.0V" and "the pack sits at 7.2V" at full charge, so VBAT runs 5.0-7.3V. Fetched from that doc, not assumed. J2 is a generic 2-pin placeholder for the board-to-board link, same treatment as J1 for th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"
