File: kicad/audio-board/audio-board.kicad_sch (KiCad schematic)
At the start: 63 parts, among them J1 TO_CM5, J2 VBAT_IN, J3 A2B_TO_CUPS, U1 ADAU1861, U10 ADP7118AUJZ-3.3-R7, U2 ADXL354CEZ, U3 LTC6242, U4 IM72D128VV01, U5 AD2428WBCPZ, U6 SN74LVC8T245PWR, U7 SN74LVC8T245PWR, U8 PCA9517ADP, U9 ADP7118AUJZ-1.8-R7

Commit message: [LIMA] audio board: clean-slate schematic from JULIETT's spec - hub, codec, AD2428, K1 bypass; netlist == design file, ERC 0 errors
Co-Authored-By: Claude Opus 5.5 <noreply@anthropic.com>
Parts:
- removed J1: TO_CM5, symbol Connector_Generic:Conn_01x11
- removed J2: VBAT_IN, symbol Connector_Generic:Conn_01x02
- removed J3: A2B_TO_CUPS, symbol Connector_Generic:Conn_01x02
- removed U1: ADAU1861, symbol AnalogDevices:ADAU1861
- removed U10: ADP7118AUJZ-3.3-R7, symbol AnalogDevices:ADP7118
- removed U2: ADXL354CEZ, symbol AnalogDevices:ADXL354
- removed U3: LTC6242, symbol AnalogDevices:LTC6242
- removed U4: IM72D128VV01, symbol Infineon:IM72D128V
- removed U5: AD2428WBCPZ, symbol AnalogDevices:AD2428
- removed U6, U7: SN74LVC8T245PWR, symbol TexasInstruments:SN74LVC8T245
- removed U8: PCA9517ADP, symbol NXP:PCA9517A
- removed U9: ADP7118AUJZ-1.8-R7, symbol AnalogDevices:ADP7118
- added C35: 1uF, symbol Device:C
- added C36: 10uF, symbol Device:C
- added C37, C43: 10uF 25V, symbol Device:C
- added C38, C40, C42, C44, C45: 100nF, symbol Device:C
- added C39, C41: 4.7uF, symbol Device:C
- added C46, C51, C54, C55, C56: 33nF, symbol Device:C
- added C47: 15nF, symbol Device:C
- added C48: 3.3nF, symbol Device:C
- added C49: 12pF C0G, symbol Device:C
- added C50: 27pF C0G, symbol Device:C
- added C52, C53: 10nF, symbol Device:C
- added D1: BAT54S, symbol Diode:BAT54S
- added D2: CDBU0130L, symbol Device:D_Schottky
- added D3: ZLLS400, symbol Device:D_Schottky
- added J1: HOST_J3 (AeroNode), symbol Connector_Generic:Conn_01x10
- added J2: HOST_J4 (AeroNode), symbol Connector_Generic:Conn_01x06
- added J3: CUP_L (A2B + speaker), symbol Connector_Generic:Conn_01x04
- added J4: CUP_R (speaker), symbol Connector_Generic:Conn_01x02
- added J5: PANEL (ear + mic), symbol Connector_Generic:Conn_01x04
- added J6: FAILSAFE_ELECTRET, symbol Connector_Generic:Conn_01x02
- added L5, L6: 180nH, symbol Device:L
- added Q1: AO3401A, symbol Transistor_FET:AO3401A
- added Q2: 2N7002, symbol Transistor_FET:2N7002
- added R10, R12: 10k 0.1%, symbol Device:R
- added R11, R13: 1k 0.1%, symbol Device:R
- added R14, R15: 10k, symbol Device:R
- added R16: 47R, symbol Device:R
- added R17: 33k, symbol Device:R
- added R18: 1R 1206, symbol Device:R
- added R19: 3.3k, symbol Device:R
- added R20: 1k, symbol Device:R
- added R21, R22: 120R, symbol Device:R
- added R23, R24: 390R, symbol Device:R
- added R25: 100k, symbol Device:R
- added R26: 0R (VDRIVE to GND: external DVDD), symbol Device:R
- added T2: Triad SP-74 (cup L), symbol Device:Transformer_1P_2S
- added T3: Triad SP-74 (cup R), symbol Device:Transformer_1P_2S
- added U1: TPS62162DSG, symbol Regulator_Switching:TPS62162DSG
- added U10: AQW612S (K1 mic-hi), symbol Panasonic:AQW612S
- added U11: AQW612S (K1 mic-lo), symbol Panasonic:AQW612S
- added U2: TPS62160DSG, symbol Regulator_Switching:TPS62160DSG
- added U3: ADP7118AUJZ-3.3-R7, symbol AnalogDevices:ADP7118
- added U4: ADAU1467, symbol AnalogDevices:ADAU1467
- added U5: W25Q32JVSS, symbol Memory_Flash:W25Q32JVSS
- added U6: ADAU1372, symbol AnalogDevices:ADAU1372
- added U7: IM68A130A, symbol Infineon:IM68A130A
- added U8: TLV9062xD, symbol Amplifier_Operational:TLV9062xD
- added U9: AD2428WBCPZ, symbol AnalogDevices:AD2428
- added Y1: SiT8008 12.288MHz 3.3V, symbol Oscillator:SiT8008xx-1x-xxE
- C1, C3: value 100nF C0G 5% -> 10uF 25V
- C10: value 1uF -> 5.6nF C0G
- C11, C12: value 0.1uF -> 100nF
- C14, C15, C16, C17, C18: value 1uF -> 100nF
- C19, C20: value 4.7uF -> 100nF
- C2: value 100nF C0G 5% -> 22uF 10V
- C22: value 10nF -> 10uF
- C23, C24, C26: value 2.2uF -> 10uF
- C25: value 2.2uF -> 1uF
- C27: value 12pF -> 1uF
- C28: value 27pF -> 10uF
- C29: value 0.033uF -> 1uF
- C30, C31: value 0.01uF -> 100nF
- C32, C33, C34: value 0.033uF -> 100nF
- C4: value 1uF -> 22uF 6.3V
- C5: value 10uF -> 2.2uF 25V
- C6: value 10uF -> 2.2uF 10V
- C7, C8: value 10uF -> 100nF
- C9: value 10uF -> 150pF C0G
- FL1: value 2600R@100MHz -> 2600R@100MHz CMC
- L1, L2: value 180nH -> 2.2uH
- R1: value 1M 1% -> 49.9k 1%
- R2: value 1M 1% -> 100k 1%
- R3: value 1M 1% -> 100k
- R4: value 2.0k -> 10k
- R5: value 2.0k -> 4.3k 1%
- R6: value 4.7k -> 100R
- R7: value 4.7k -> 10k
- R8: value 120R -> 10k
- R9: value 120R -> 0R
Connections:
- net A2B_BIAS_P is gone; now on net A2B_LINE_P: L3.2
- net ACCEL_V1P8DIG is gone; now on net +3V3A: C17.1
- net CM is gone; now on net +1V2: C4.1
- net X_ACCEL_OUT is gone; now on net VBAT: C1.1
- net Y_ACCEL_OUT is gone; now on net +3V3: C2.1
- net Z_ACCEL_OUT is gone; now on net VBAT: C3.1
- net A2B_BCM: now also U9.24 (BCM)
- net A2B_BN: now also C49.2, L6.1, U9.23 (BN); no longer C27.2, L2.1
- net A2B_BP: now also C49.1, L5.1, U9.22 (BP); no longer C27.1, L1.1
- net A2B_LINE_N: now also C53.2, C55.1, C56.2, J3.2 (Pin_2); no longer C31.2, C33.1, C34.2
- net A2B_LINE_P: now also C52.2, C54.1, C56.1, J3.1 (Pin_1); no longer C30.2, C32.1, C34.1, L3.1
- net A2B_VOUT1: now also C39.1, C40.1, U9.1 (PLLVDD), U9.2 (DVDD), U9.3 (DVDD), U9.32 (VOUT1); no longer C19.1
- net A2B_VOUT2: now also C41.1, C42.1, U9.20 (ATRXVDD), U9.21 (BTRXVDD), U9.29 (VOUT2); no longer C20.1, C21.1, C22.1
- net VBAT: now also C5.1, D2.2 (A), D3.2 (A), J1.10 (Pin_10), R23.1, R24.1, U1.2 (VIN), U1.3 (EN), U2.2 (VIN), U3.1 (VIN), U3.3 (EN); no longer C24.1, C26.1
- net 1V8 renamed +3V3
- net +3V3: now also C13.1, C14.1, C15.1, C34.1, L1.2, R3.1, C45.1, U1.6 (VOS), U2.3 (EN), U4.2 (IOVDD), U4.22 (IOVDD), U4.37 (IOVDD), U4.46 (IOVDD), U4.68 (IOVDD), U5.3 (~{WP}/IO_{2}), U5.7 (~{HOLD}/~{RESET}/IO_{3}), U5.8 (VCC), U6.40 (IOVDD), U9.9 (IOVDD), Y1.1 (OE), Y1.4 (Vdd); no longer C10.1, C18.1, C5.1, C6.1, C9.1, R5.1
- removed net 3V3_ACCEL: C13.1, C14.1, C15.1, C25.1, R6.1, R7.1
- net A2B_BIAS_N renamed A2B_VSSN
- net A2B_VSSN: now also U9.26 (VSSN)
- net A2B_BN_F renamed +1V2
- net +1V2: now also C18.1, C19.1, C20.1, C21.1, C22.1, R1.1, U2.6 (VOS), U4.24 (DVDD), U4.43 (DVDD), U4.65 (DVDD), U4.87 (DVDD); no longer FL1.3
- removed net A2B_BN_T: C31.1, FL1.4, R9.2
- removed net A2B_BP_F: C28.1, FL1.1, L1.2
- removed net A2B_BP_T: C30.1, FL1.2, R8.1
- removed net A2B_TERM_CT: C29.1, R8.2, R9.1
- net ACCEL_V1P8ANA renamed +3V3A
- net +3V3A: now also C10.1, C31.1, C32.1, C33.1, C6.1, C9.1, R6.1, C38.1, D1.2 (K), R14.1, U3.4 (SENSE/ADJ), U3.5 (VOUT), U4.19 (PVDD), U4.9 (AVDD), U6.10 (AVDD), U6.19 (AVDD), U6.24 (AVDD), U8.8 (V+)
- net AGND renamed GND
- net GND: now also C1.2, C2.2, C3.2, C30.2, C31.2, C34.2, R2.2, R8.2, R9.2, C35.2, C36.2, C38.2, C39.2, C40.2, C41.2, C42.2, C43.2, C44.2, C45.2, C46.2, C50.2, C51.2, C54.2, C55.2, D1.1 (A), J1.1 (Pin_1), Q2.2 (S), R15.2, R25.2, R26.2, U1.1 (PGND), U1.4 (AGND), U1.5 (FB), U1.9 (PAD), U11.5 (NO), U2.1 (PGND), U2.4 (AGND), U2.9 (PAD), U3.2 (GND), U4.1 (DGND), U4.18 (PGND), U4.21 (DGND), U4.23 (DGND), U4.29 (DGND), U4.36 (DGND), U4.40 (MOSI/ADDR1), U4.41 (~{SS}/ADDR0), U4.44 (DGND), U4.45 (DGND), U4.66 (DGND), U4.67 (DGND), U4.8 (AGND), U4.88 (DGND), U4.89 (EP), U5.4 (GND), U6.11 (AGND), U6.20 (AGND), U6.23 (AGND), U6.3 (ADDR1/MOSI), U6.30 (DGND), U6.4 (ADDR0/SS), U6.41 (EP), U6.5 (DGND), U7.2 (GND), U7.4 (GND), U8.4 (V-), U9.25 (VSS), U9.31 (VSS), U9.33 (EPAD), U9.7 (ADR1/IO1), U9.8 (ADR2/IO2), Y1.2 (GND); no longer C10.2, C25.2, C9.2
- removed net CM_BUF: R1.2, R2.2, R3.2
- net SCL renamed SELFBOOT
- net SELFBOOT: now also U4.42 (SELFBOOT)
- net SCL_3V3 renamed MIC_VDD
- net MIC_VDD: now also C35.1, U7.3 (VDD)
- net SDA renamed PLLFILT
- net PLLFILT: now also C9.2, U4.20 (PLLFILT)
- net SDA_3V3 renamed COMMS_TAP
- net COMMS_TAP: now also C27.1, R8.1
- removed net X_COUPLE: C1.2, R1.1
- net Y_COUPLE renamed FB1V2
- net FB1V2: now also R1.2, U2.5 (FB); no longer C2.2
- removed net Z_COUPLE: C3.2, R3.1
- new net A2B_BCLK: U4.59 (BCLK_OUT3), U4.84 (BCLK_IN3), U9.10 (BCLK)
- new net A2B_BIASP: C48.2, L3.1, Q1.3 (D), R20.1
- new net A2B_BNF: FL1.3, L6.2
- new net A2B_BNT: C53.1, FL1.4, R22.2
- new net A2B_BPF: C50.1, FL1.1, L5.2
- new net A2B_BPT: C52.1, FL1.2, R21.1
- new net A2B_DRX0: U4.60 (SDATA_OUT3), U9.14 (DRX0/IO5)
- new net A2B_DRX1: U4.64 (SDATAIO4/MP20), U9.15 (DRX1/IO6)
- new net A2B_DTX0: U4.86 (SDATA_IN3), U9.12 (DTX0/IO3)
- new net A2B_DTX1: U4.63 (SDATAIO5/MP21), U9.13 (DTX1/IO4)
- new net A2B_GATE: C47.2, C48.1, Q1.1 (G), R17.2, R19.2
- new net A2B_IRQ: J2.2 (Pin_2), U9.6 (IRQ/IO0)
- new net A2B_QS: Q1.2 (S), R18.2
- new net A2B_SENSE: R20.2, U9.28 (SENSE)
- new net A2B_SWP: R19.1, U9.27 (SWP)
- new net A2B_SYNC: U4.58 (LRCLK_OUT3/MP9), U4.85 (LRCLK_IN3/MP13), U9.11 (SYNC)
- new net A2B_TCT: C51.1, R21.2, R22.1
- new net A2B_VIN: C43.1, C44.1, D2.1 (K), U9.30 (VIN)
- new net A2B_VPWR: C46.1, C47.1, D3.1 (K), R17.1, R18.1
- new net AIN0: C25.2, U6.9 (AIN0)
- new net AIN0REF: C24.1, U6.8 (AIN0REF)
- new net AIN1: C27.2, D1.3 (COM), U6.14 (AIN1)
- new net AIN1REF: C26.1, U6.13 (AIN1REF)
- new net BOOT_CS: U4.32 (~{SS_M}/MP0), U5.1 (~{CS})
- new net BOOT_MISO: U4.35 (SDA_M/MISO_M/MP3), U5.2 (DO/IO_{1})
- new net BOOT_MOSI: U4.33 (MOSI_M/MP1), U5.5 (DI/IO_{0})
- new net BOOT_SCLK: U4.34 (SCL_M/SCLK_M/MP2), U5.6 (CLK)
- new net CABIN_MIC: C25.1, U7.1 (OUT)
- new net CODEC_ADC: U4.83 (SDATA_IN2), U6.34 (ADC_SDATA0/MP1)
- new net CODEC_BCLK: U4.56 (BCLK_OUT2), U4.81 (BCLK_IN2), U6.32 (BCLK)
- new net CODEC_CM: C28.1, U6.12 (CM)
- new net CODEC_DAC: U4.57 (SDATA_OUT2), U6.33 (DAC_SDATA/MP0)
- new net CODEC_DVDD: C29.1, C30.1, U6.28 (REG_OUT), U6.29 (DVDD)
- new net CODEC_LRCLK: U4.55 (LRCLK_OUT2/MP8), U4.82 (LRCLK_IN2/MP12), U6.31 (LRCLK)
- new net CODEC_MCLK: U4.27 (CLKOUT), U6.39 (XTALI/MCLKIN)
- new net CTL_MIC: J2.1 (Pin_1), Q2.1 (G), R25.1
- new net DAC_N: R12.1, U6.21 (HPOUTLN/LOUTLN)
- new net DAC_P: R10.1, U6.22 (HPOUTLP/LOUTLP)
- new net EAR_HI: J5.1 (Pin_1), T2.1 (AA), T3.1 (AA)
- new net EAR_RTN: J5.2 (Pin_2), T2.2 (AB), T3.2 (AB)
- new net ELEC_HI: J6.1 (Pin_1), U10.7 (NC)
- new net ELEC_LO: J6.2 (Pin_2), U11.7 (NC)
- new net HOST_SDI0: J1.4 (Pin_4), U4.49 (SDATA_OUT0)
- new net HOST_SDI1: J1.6 (Pin_6), U4.52 (SDATA_OUT1)
- new net HOST_SDI2: J2.3 (Pin_3), U4.72 (SDATAIO0/MP16)
- new net HOST_SDI3: J2.5 (Pin_5), U4.70 (SDATAIO2/MP18)
- new net HOST_SDO0: J1.5 (Pin_5), U4.75 (SDATA_IN0)
- new net HOST_SDO1: J1.7 (Pin_7), U4.78 (SDATA_IN1)
- new net HOST_SDO2: J2.4 (Pin_4), U4.71 (SDATAIO1/MP17)
- new net HOST_SDO3: J2.6 (Pin_6), U4.69 (SDATAIO3/MP19)
- new net I2C_SCL: J1.8 (Pin_8), U4.39 (SCLK/SCL), U6.2 (SCL/SCLK), U9.4 (SCL)
- new net I2C_SDA: J1.9 (Pin_9), U4.38 (MISO/SDA), U6.1 (SDA/MISO), U9.5 (SDA)
- new net I2S_BCLK: J1.3 (Pin_3), U4.48 (BCLK_OUT0), U4.73 (BCLK_IN0)
- new net I2S_WS: J1.2 (Pin_2), U4.47 (LRCLK_OUT0/MP4), U4.74 (LRCLK_IN0/MP10)
- new net K1A_LED: R23.2, U10.1 (NC_LED_A)
- new net K1A_MID: U10.2 (NC_LED_K), U10.3 (NO_LED_A)
- new net K1B_LED: R24.2, U11.1 (NC_LED_A)
- new net K1B_MID: U11.2 (NC_LED_K), U11.3 (NO_LED_A)
- new net K1_DRV: Q2.3 (D), U10.4 (NO_LED_K), U11.4 (NO_LED_K)
- new net MCLK_IN: U4.25 (XTALIN/MCLK), Y1.3 (OUT)
- new net MIC_HI: J5.3 (Pin_3), U10.6 (NO), U10.8 (NC)
- new net MIC_LO: J5.4 (Pin_4), U11.6 (NO), U11.8 (NC)
- new net OPA_INN: R12.2, R13.1, U8.2 (-)
- new net OPA_INP: R10.2, R11.1, U8.3 (+)
- new net PLL_RC: C10.2, R5.1
- new net PV_BUF: C37.1, R13.2, U8.1
- new net PV_C: C37.2, R16.1
- new net PV_OUT: R16.2, U10.5 (NO)
- new net RESET_N: R3.2, U2.8 (PG), U4.28 (~{RESET}), U6.27 (PD)
- new net SPK_L_A: J3.3 (Pin_3), R7.1, T2.3 (SA), T2.5 (SC)
- new net SPK_L_B: J3.4 (Pin_4), R9.1, T2.4 (SB), T2.6 (SD)
- new net SPK_R_A: J4.1 (Pin_1), T3.3 (SA), T3.5 (SC)
- new net SPK_R_B: J4.2 (Pin_2), T3.4 (SB), T3.6 (SD)
- new net SW1V2: L2.1, U2.7 (SW)
- new net SW3V3: L1.1, U1.7 (SW)
- new net U8B_FB: U8.6 (-), U8.7
- new net VDRIVE: R26.1, U4.3 (VDRIVE)
- new net VREF_MID: C36.1, R11.2, R14.2, R15.1, U8.5 (+)
- no-connect marks 16 -> 42
Other:
- removed sheet AIRCRAFT AUDIO I/O
- note added: "A2B MAIN NODE: AD2428 (ruling 9), circuit per EVAL-AD2428WD1BZ sheet 2, B side VIN from VBAT via D2 (VIN 3.7-9.0 V). Bus power: VBAT -> D3 -> R18 -> Q1 (gate: SWP via R19) -> L3 -> line +. Line - -> L4 -> VSSN (internal switch, 300 mA). SENSE reads the switched bias via R20. Coupling: FB1/FB2 to BCM, C49, L5/L6, C50, FL1 CMC, R21/R22 + C51, C52/C53 series, C54-C56. Cups daisy-chain J3 -> cup L ->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"
- note added: "AIRCRAFT / BYPASS: aircraft-powered whenever we are off T2/T3 Triad SP-74: primaries in parallel on the panel earphone line, secondaries paralleled (3/5, 4/6). K1 = U10 (mic-hi) + U11 (mic-lo), AQW612S each (ruling 2). LEDs OFF = bypass: electret J6 -> panel mic. CTL_MIC high -> Q2 on -> LEDs on (VBAT via R23/R24 390R, 5.1-12.8 mA) -> Form A: PV_OUT / GND -> panel. Watchdog parked (ruling 4): a h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"
- note added: "CODEC: ADAU1372 ADC0 = cabin mic U7 IM68A130A, single-ended analogue (John, 2026-10-21), from 3V3A via R6/C35. ADC1 = comms tap off the T2 secondary: R7/R8 10k/10k, C27, BAT54S D1 clamp to the rails. DAC0 (HPOUTL +/-) -> U8A difference amp, gain 0.1 about VREF_MID -> C37 / R16 -> PV_OUT -> K1 Form A. Panel mic input level is unspecified (spec section 9): gain set by R10-R13, trim in DSP."
- note added: "HUB: ADAU1467 (clock master, routing, CM5 I/O) One 12.288 MHz XO into XTALIN/MCLK; hub drives CODEC_MCLK (CLKOUT) and every BCLK/LRCLK. Self-boot from U5 W25Q32 on the SPI master (SPI mode 3, read 0x03). I2C slave, ADDR1/ADDR0 = 0. PLL filter per DS Fig. 16 (150 pF || 5.6 nF + 4.3 k, to PVDD). VDRIVE to GND via R26: DVDD is external. OUT0/IN0 = CM5, OUT2/IN2 = codec, OUT3/IN3 + SDATAIO4/5 = A2B, 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"
- note added: "POWER + HOST HEADER VBAT = AeroNode BAT_PWR: 2S LiFePO4, 5.0-7.3 V [repo, not confirmed on the AeroNode sheet]. U1 3V3 buck (I/O) / U2 1V2 buck (hub core 330 mA typ, 940 mA max; TPS62160 is 1 A) / U3 3V3A LDO. U2 PG = RESET_N for hub + codec. J1/J2 mirror AeroNode J3/J4 pin-for-pin (2026-08-31 sheet). CM5 = I2S consumer (rp1_i2s1), max 8 ch, 32-bit. HOST_SDO1 = coefficient lane (ruling 8). CTL_MI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"
- note removed: "A2B LINE INTERFACE - U5 B-side, to the earcups Values TRANSCRIBED from ADI's own master-node eval board, EVAL-AD2428WD1BZ Rev 1.1 sheet 2 of 7 (archived in docs/datasheets, pinned in fetch-datasheets.sh). An eval board is NOT ADI's issued recommendation - AD242x Rev. C p.33 makes that distinction decide automotive-grade compliance. REVIEW WITH ADI BEFORE FAB. A2B_BIAS_P has NO SOURCE yet - the bu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"
- note removed: "HPOUTN intentionally left no-connect (corrected back, 2026-09-29 - this sheet briefly used both HPOUTP/HPOUTN differentially into the BOOM MIC / TX SELECT sheet's transformer, then reverted to single-ended HPOUTP only). A series blocking cap on that sheet now handles what the differential connection used to handle for free: HPOUTP sits at the DAC's ~0.85V common-mode bias, and driving a transform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"
- note removed: "I2S + I2C crossing to the host (CM5/RP1), per docs/audio-board-level-shifter.md (this note's "1860" is the same silicon as our 1861, UG-2257 p.1) and Decision D in docs/audio-board-decision-record.md. SIX signals now cross to the host, on TWO I2S/TDM lanes sharing ONE clock pair: BCLK_0, FSYNC_0, SDATAO_0, and NOW U5's DTX0 go UP through U6 (SN74LVC8T245, DIR=1V8 so A->B, using the two channels f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"
- note removed: "PRELIM - ADXL354 single-ended front end into the ADAU1861. Per docs/sensor-head-design-note.md and docs/audio-board-decision-record.md (Decision B: ADAU1861 ruled, ADAU1372 rejected for this board). WIRED: ADAU1861 full power tree (1V8/AGND) + boot straps (PD, SELFBOOT, ROM_BOOT_MODE, REG_EN - tied to safe defaults, [assumed], not checked against UG-2257's boot section yet). ADXL354 X/Y/Z -> 100n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"
- note removed: "Power in: VBAT from the aeronode board (U9/U10, J2). This is the ONLY supply arriving on this board - Peter confirmed no 3.3V rail comes over from the CM5 side at all. VBAT is aeronode's raw 2S LiFePO4 pack net (ahead of its charger/buck stage) - per kicad/aeronode/doc/ARCHITECTURE.md: "the pack never falls below 5.0V" and "the pack sits at 7.2V" at full charge, so VBAT runs 5.0-7.3V. Fetched fro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"

Commit message: [LIMA] audio board: ruling 10 drawn - T4 SM-LP-5001 replaces the TLV9062 buffer; mic return isolated from GND
Co-Authored-By: Claude Opus 5.5 <noreply@anthropic.com>
Parts:
- removed C36: 10uF, symbol Device:C
- removed C38: 100nF, symbol Device:C
- removed R11, R13: 1k 0.1%, symbol Device:R
- removed R12: 10k 0.1%, symbol Device:R
- removed R14, R15: 10k, symbol Device:R
- removed R16: 47R, symbol Device:R
- removed U8: TLV9062xD, symbol Amplifier_Operational:TLV9062xD
- added T4: Bourns SM-LP-5001 (600:600), symbol Device:Transformer_1P_1S
- C37: value 10uF 25V -> 220nF film
- R10: value 10k 0.1% -> 10k
Connections:
- net PV_BUF is gone; now on net PV_ATT: C37.1
- net PV_C is gone; now on net PV_OUT: C37.2
- net DAC_N: now also T4.2 (AB)
- net DAC_P: now also T4.1 (AA); no longer R10.1
- net GND: no longer U11.5 (NO)
- net OPA_INP renamed PV_ATT
- new net PV_RTN: T4.4 (SB), U11.5 (NO)
- new net PV_SEC: R10.1, T4.3 (SA)
Other:
- note added: "AIRCRAFT / BYPASS: aircraft-powered whenever we are off T2/T3 Triad SP-74: primaries in parallel on the panel earphone line, secondaries paralleled (3/5, 4/6). K1 = U10 (mic-hi) + U11 (mic-lo), AQW612S each (ruling 2). LEDs OFF = bypass: electret J6 -> panel mic. CTL_MIC high -> Q2 on -> LEDs on (VBAT via R23/R24 390R, 5.1-12.8 mA) -> Form A: PV_OUT / PV_RTN (T4) -> panel. Both mic legs stay isol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"
- note added: "CODEC: ADAU1372 ADC0 = cabin mic U7 IM68A130A, single-ended analogue (John, 2026-10-21), from 3V3A via R6/C35. ADC1 = comms tap off the T2 secondary: R7/R8 10k/10k, C27, BAT54S D1 clamp (ADC FS 0.90 Vrms). DAC0 (HPOUTL +/-, 1.94 Vrms diff FS) drives T4 SM-LP-5001 primary directly (ruling 10). T4 secondary (aircraft side) -> R10 10k -> C37 220 nF film -> PV_OUT -> K1 Form A; return PV_RTN -> K1 mi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"
- note removed: "AIRCRAFT / BYPASS: aircraft-powered whenever we are off T2/T3 Triad SP-74: primaries in parallel on the panel earphone line, secondaries paralleled (3/5, 4/6). K1 = U10 (mic-hi) + U11 (mic-lo), AQW612S each (ruling 2). LEDs OFF = bypass: electret J6 -> panel mic. CTL_MIC high -> Q2 on -> LEDs on (VBAT via R23/R24 390R, 5.1-12.8 mA) -> Form A: PV_OUT / GND -> panel. Watchdog parked (ruling 4): a h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"
- note removed: "CODEC: ADAU1372 ADC0 = cabin mic U7 IM68A130A, single-ended analogue (John, 2026-10-21), from 3V3A via R6/C35. ADC1 = comms tap off the T2 secondary: R7/R8 10k/10k, C27, BAT54S D1 clamp to the rails. DAC0 (HPOUTL +/-) -> U8A difference amp, gain 0.1 about VREF_MID -> C37 / R16 -> PV_OUT -> K1 Form A. Panel mic input level is unspecified (spec section 9): gain set by R10-R13, trim in DSP."
- moved on the sheet: R10

Commit message: [LIMA] audio board: ruling 11 - CTL_SPKR to AD2428 IO7 for cup K2 via GPIO-over-distance; A2B IRQ dropped
Co-Authored-By: Claude Opus 5.5 <noreply@anthropic.com>
Connections:
- net CTL_SPKR: now reaches U9.16 (PDMCLK/IO7)
- net CTL_SPKR: now also J2.2 (Pin_2)
- net A2B_IRQ: no longer names the net of U9.6 (IRQ/IO0)
- net A2B_IRQ: no longer J2.2 (Pin_2)
Changed lines of the file:
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@@
 	)
 	(no_connect
-		(at 589.28 453.39)
-	)
-	(no_connect
 		(at 548.64 430.53)
 	)
@@
 		(at 548.64 435.61)
 	)
-	(text "POWER + HOST HEADER\nVBAT = AeroNode BAT_PWR: 2S LiFePO4, 5.0-7.3 V [repo, not confirmed on the AeroNode sheet].\nU1 3V3 buck (I/O) / U2 1V2 buck (hub core 330 mA typ, 940 mA max; TPS62160 is 1 A) / U3 3V3A LDO.\nU2 PG = RESET_N for hub + codec. J1/J2 mirror AeroNode J3/J4 pin-for-pin (2026-08-31 sheet).\nCM5 = I2S consumer (rp1_i2s1), max 8 ch, 32-bit. HOST_SDO1 = coefficient lane (ruling 8).\nCTL_MIC drives K1. CTL_SPKR is re-used as A2B_IRQ."
-		(at 95.25 25.4 0)
+	(no_connect
+		(at 589.28 430.53)
+	)
+	(text "HUB: ADAU1467 (clock master, routing, CM5 I/O)\nOne 12.288 MHz XO into XTALIN/MCLK; hub drives CODEC_MCLK (CLKOUT) and every BCLK/LRCLK.\nSelf-boot from U5 W25Q32 on the SPI master (SPI mode 3, read 0x03). I2C slave, ADDR1/ADDR0 = 0.\nPLL filter per DS Fig. 16 (150 pF || 5.6 nF + 4.3 k, to PVDD). VDRIVE to GND via R26: DVDD is external.\nOUT0/IN0 = CM5, OUT2/IN2 = codec, OUT3/IN3 + SDATAIO4/5 = A2B, SDATAIO0-3 = spare CM5 lanes.\nThe coefficient channel must be routed bit-exact: no ASRC, gain, mix or dither."
+		(at 365.76 93.98 0)
 		(effects
 			(font
@@
 		)
 	)
-	(text "HUB: ADAU1467 (clock master, routing, CM5 I/O)\nOne 12.288 MHz XO into XTALIN/MCLK; hub drives CODEC_MCLK (CLKOUT) and every BCLK/LRCLK.\nSelf-boot from U5 W25Q32 on the SPI master (SPI mode 3, read 0x03). I2C slave, ADDR1/ADDR0 = 0.\nPLL filter per DS Fig. 16 (150 pF || 5.6 nF + 4.3 k, to PVDD). VDRIVE to GND via R26: DVDD is external.\nOUT0/IN0 = CM5, OUT2/IN2 = codec, OUT3/IN3 + SDATAIO4/5 = A2B, SDATAIO0-3 = spare CM5 lanes.\nThe coefficient channel must be routed bit-exact: no ASRC, gain, mix or dither."
-		(at 365.76 93.98 0)
+	(text "A2B MAIN NODE: AD2428 (ruling 9), circuit per EVAL-AD2428WD1BZ sheet 2, B side\nVIN from VBAT via D2 (VIN 3.7-9.0 V). Bus power: VBAT -> D3 -> R18 -> Q1 (gate: SWP via R19) -> L3 -> line +.\nLine - -> L4 -> VSSN (internal switch, 300 mA). SENSE reads the switched bias via R20.\nCoupling: FB1/FB2 to BCM, C49, L5/L6, C50, FL1 CMC, R21/R22 + C51, C52/C53 series, C54-C56.\nCups daisy-chain J3 -> cup L -> cup R. OPEN: bus-power margin at 5.0 V through two cups."
+		(at 637.54 320.04 0)
 		(effects
 			(font
@@
 		)
 	)
-	(text "A2B MAIN NODE: AD2428 (ruling 9), circuit per EVAL-AD2428WD1BZ sheet 2, B side\nVIN from VBAT via D2 (VIN 3.7-9.0 V). Bus power: VBAT -> D3 -> R18 -> Q1 (gate: SWP via R19) -> L3 -> line +.\nLine - -> L4 -> VSSN (internal switch, 300 mA). SENSE reads the switched bias via R20.\nCoupling: FB1/FB2 to BCM, C49, L5/L6, C50, FL1 CMC, R21/R22 + C51, C52/C53 series, C54-C56.\nCups daisy-chain J3 -> cup L -> cup R. OPEN: bus-power margin at 5.0 V through two cups."
-		(at 637.54 320.04 0)
+	(text "CODEC: ADAU1372\nADC0 = cabin mic U7 IM68A130A, single-ended analogue (John, 2026-10-21), from 3V3A via R6/C35.\nADC1 = comms tap off the T2 secondary: R7/R8 10k/10k, C27, BAT54S D1 clamp (ADC FS 0.90 Vrms).\nDAC0 (HPOUTL +/-, 1.94 Vrms diff FS) drives T4 SM-LP-5001 primary directly (ruling 10).\nT4 secondary (aircraft side) -> R10 10k -> C37 220 nF film -> PV_OUT -> K1 Form A; return PV_RTN -> K1 mic-lo.\nAbout 69 mVrms into a ~470 ohm mic input at 0 dBFS [derived; panel input spec unknown]. No path to our GND."
+		(at 609.6 25.4 0)
+		(effects
+			(font
+				(size 1.778 1.778)
+			)
+		)
+	)
+	(text "AIRCRAFT / BYPASS: aircraft-powered whenever we are off\nT2/T3 Triad SP-74: primaries in parallel on the panel earphone line, secondaries paralleled (3/5, 4/6).\nK1 = U10 (mic-hi) + U11 (mic-lo), AQW612S each (ruling 2). LEDs OFF = bypass: electret J6 -> panel mic.\nCTL_MIC high -> Q2 on -> LEDs on (VBAT via R23/R24 390R, 5.1-12.8 mA) -> Form A: PV_OUT / PV_RTN (T4) -> panel.\nBoth mic legs stay isolated from our GND in both states. Watchdog parked (ruling 4). SP-74 polarity unverified."
+		(at 132.08 370.84 0)
 		(effects
 			(font
@@
 		)
 	)
-	(label "A2B_IRQ"
-		(at 25.4 116.84 180)
-		(effects
-			(font
-				(size 1.27 1.27)
-			)
-			(justify right bottom)
-		)
-	)
-	(label "A2B_IRQ"
-		(at 589.28 430.53 0)
-		(effects
-			(font
-				(size 1.27 1.27)
-			)
-			(justify left bottom)
-		)
-	)
 	(label "HOST_SDI2"
 		(at 25.4 119.38 180)
@@
 		)
 	)
-  (label "DAC_P"
-    (at 650.24 274.32 180)
-    (fields_autoplaced yes)
-    (effects (font (size 1.27 1.27)) (justify right bottom))
-  )
-  (label "DAC_N"
-    (at 650.24 284.47999999999996 180)
+	(label "DAC_P"
+		(at 650.24 274.32 180)
+		(effects
+			(font
+				(size 1.27 1.27)
+			)
+			(justify right bottom)
+		)
+	)
+	(label "DAC_N"
+		(at 650.24 284.48 180)
+		(effects
+			(font
+				(size 1.27 1.27)
+			)
+			(justify right bottom)
+		)
+	)
+	(label "PV_SEC"
+		(at 670.56 284.48 0)
+		(effects
+			(font
+				(size 1.27 1.27)
+			)
+			(justify left bottom)
+		)
+	)
+	(label "PV_SEC"
+		(at 693.42 273.05 0)
+		(effects
+			(font
+				(size 1.27 1.27)
+			)
+			(justify left bottom)
+		)
+	)
+	(label "PV_ATT"
+		(at 693.42 280.67 0)
+		(effects
+			(font
+				(size 1.27 1.27)
+			)
+			(justify left bottom)
+		)
+	)
+	(label "PV_ATT"
+		(at 726.44 295.91 0)
+		(effects
+			(font
+				(size 1.27 1.27)
+			)
+			(justify left bottom)
+		)
+	)
+	(label "PV_OUT"
+		(at 726.44 303.53 0)
+		(effects
+			(font
+				(size 1.27 1.27)
+			)
+			(justify left bottom)
+		)
+	)
+	(label "PV_RTN"
+		(at 670.56 274.32 0)
+		(effects
+			(font
+				(size 1.27 1.27)
+			)
+			(justify left bottom)
+		)
+	)
+	(label "PV_RTN"
+		(at 200.66 476.25 0)
+		(effects
+			(font
+				(size 1.27 1.27)
+			)
+			(justify left bottom)
+		)
+	)
+  (label "CTL_SPKR"
+    (at 25.4 116.83999999999999 180)
     (fields_autoplaced yes)
     (effects (font (size 1.27 1.27)) (justify right bottom))
   )
-  (label "PV_SEC"
-    (at 670.56 284.47999999999996 0)
-    (fields_autoplaced yes)
-    (effects (font (size 1.27 1.27)) (justify left bottom))
-  )
-  (label "PV_SEC"
-    (at 693.42 273.05 0)
-    (fields_autoplaced yes)
-    (effects (font (size 1.27 1.27)) (justify left bottom))
-  )
-  (label "PV_ATT"
-    (at 693.42 280.67 0)
-    (fields_autoplaced yes)
-    (effects (font (size 1.27 1.27)) (justify left bottom))
-  )
-  (label "PV_ATT"
-    (at 726.44 295.91 0)
+  (label "CTL_SPKR"
+    (at 589.2800000000001 453.39000000000004 0)
     (fields_autoplaced yes)
     (effects (font (size 1.27 1.27)) (justify left bottom))
   )
-  (label "PV_OUT"
-    (at 726.44 303.53000000000003 0)
-    (fields_autoplaced yes)
-    (effects (font (size 1.27 1.27)) (justify left bottom))
-  )
-  (label "PV_RTN"
-    (at 670.56 274.32 0)
-    (fields_autoplaced yes)
-    (effects (font (size 1.27 1.27)) (justify left bottom))
-  )
-  (label "PV_RTN"
-    (at 200.66 476.25 0)
-    (fields_autoplaced yes)
-    (effects (font (size 1.27 1.27)) (justify left bottom))
-  )
-  (text "CODEC: ADAU1372\nADC0 = cabin mic U7 IM68A130A, single-ended analogue (John, 2026-10-21), from 3V3A via R6/C35.\nADC1 = comms tap off the T2 secondary: R7/R8 10k/10k, C27, BAT54S D1 clamp (ADC FS 0.90 Vrms).\nDAC0 (HPOUTL +/-, 1.94 Vrms diff FS) drives T4 SM-LP-5001 primary directly (ruling 10).\nT4 secondary (aircraft side) -> R10 10k -> C37 220 nF film -> PV_OUT -> K1 Form A; return PV_RTN -> K1 mic-lo.\nAbout 69 mVrms into a ~470 ohm mic input at 0 dBFS [derived; panel input spec unknown]. No path to our GND."
-    (at 609.6 25.4 0)
-    (effects (font (size 1.778 1.778)))
-  )
-  (text "AIRCRAFT / BYPASS: aircraft-powered whenever we are off\nT2/T3 Triad SP-74: primaries in parallel on the panel earphone line, secondaries paralleled (3/5, 4/6).\nK1 = U10 (mic-hi) + U11 (mic-lo), AQW612S each (ruling 2). LEDs OFF = bypass: electret J6 -> panel mic.\nCTL_MIC high -> Q2 on -> LEDs on (VBAT via R23/R24 390R, 5.1-12.8 mA) -> Form A: PV_OUT / PV_RTN (T4) -> panel.\nBoth mic legs stay isolated from our GND in both states. Watchdog parked (ruling 4). SP-74 polarity unverified."
-    (at 132.08 370.84 0)
+  (text "POWER + HOST HEADER\nVBAT = AeroNode BAT_PWR: 2S LiFePO4, 5.0-7.3 V [repo, not confirmed on the AeroNode sheet].\nU1 3V3 buck (I/O) / U2 1V2 buck (hub core 330 mA typ, 940 mA max; TPS62160 is 1 A) / U3 3V3A LDO.\nU2 PG = RESET_N for hub + codec. J1/J2 mirror AeroNode J3/J4 pin-for-pin (2026-08-31 sheet).\nCM5 = I2S consumer (rp1_i2s1), max 8 ch, 32-bit. HOST_SDO1 = coefficient lane (ruling 8).\nCTL_MIC drives K1. CTL_SPKR -> AD2428 IO7 -> GPIO-over-distance -> cup K2 (ruling 11). A2B IRQ unused: CM5 polls."
+    (at 95.25 25.4 0)
     (effects (font (size 1.778 1.778)))
   )

Commit message: [LIMA] ruling 12: 8 V A2B bus boost (LM2731X) on the audio board; cup R7/R8 680R
Co-Authored-By: Claude Opus 5.5 <noreply@anthropic.com>
Parts:
- added C57: 10uF 16V, symbol Device:C
- added C58, C59: 10uF 25V, symbol Device:C
- added C60: 330pF, symbol Device:C
- added D4: MBR0520, symbol Device:D_Schottky
- added L7: 10uH 1.5A, symbol Device:L
- added R27: 73.2k 1%, symbol Device:R
- added R28: 13.3k 1%, symbol Device:R
- added U12: LM2731XMF (8 V A2B bus), symbol Regulator_Switching:LM2731XMF
Connections:
- net GND: now also C57.2, C58.2, C59.2, R28.2, U12.2 (GND)
- net VBAT: now also C57.1, L7.1, U12.4 (EN), U12.5 (VIN); no longer D2.2 (A), D3.2 (A)
- new net BOOST_FB: C60.2, R27.2, R28.1, U12.3 (FB)
- new net BOOST_SW: D4.2 (A), L7.2, U12.1 (SW)
- new net VBUS8: C58.1, C59.1, C60.1, D2.2 (A), D3.2 (A), D4.1 (K), R27.1
Other:
- note added: "A2B MAIN NODE: AD2428 (ruling 9), circuit per EVAL-AD2428WD1BZ sheet 2, B side VBUS8 = U12 LM2731X boost from VBAT, 8.00 V (R27/R28, Cf C60) - ruling 12, docs/a2b-bus-power-budget.md. VIN = VBUS8 via D2 (7.6 V, max 9.0). Bus power: VBUS8 -> D3 -> R18 -> Q1 (gate: SWP via R19) -> L3 -> line +. Line - -> L4 -> VSSN (internal switch, 300 mA; cups need ~188 mA worst). SENSE via R20. A2B_SWCTL.MODE = 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"
- note removed: "A2B MAIN NODE: AD2428 (ruling 9), circuit per EVAL-AD2428WD1BZ sheet 2, B side VIN from VBAT via D2 (VIN 3.7-9.0 V). Bus power: VBAT -> D3 -> R18 -> Q1 (gate: SWP via R19) -> L3 -> line +. Line - -> L4 -> VSSN (internal switch, 300 mA). SENSE reads the switched bias via R20. Coupling: FB1/FB2 to BCM, C49, L5/L6, C50, FL1 CMC, R21/R22 + C51, C52/C53 series, C54-C56. Cups daisy-chain J3 -> cup L ->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"

Commit message: [LIMA] audio board: footprints drawn and assigned (117/117)
Peter 2026-10-23: 4-layer, 0603 passives, JLCPCB assembly, JST GH for all
off-board connectors, outline mine to propose.

New footprints, via Konnect, each from its data sheet drawing:
- ADAU1467 CP-88-10 (12x12, P0.5, EP5.3) and ADAU1372 CP-40-10 (6x6, EP4.3)
- IM68A130A PG-TLGA-4-2 (plated 0.6 mm port in 1.65 mm GND ring)
- AQW612S GU SOP8, Triad SP-74 THT, Bourns SM-LP-5001
  (pads renumbered to Device:Transformer_1P_1S; terms 2/5 NC)
Courtyards/fab outlines corrected to body size (Konnect took body_height as Y).

Checked: netlist == doc/design_nets.py, ERC 0 errors (4 strap warnings),
every symbol pin has a pad in its footprint (117 parts, 0 mismatches).

Co-Authored-By: Claude Opus 5.5 <noreply@anthropic.com>
Parts:
- C1, C2, C22, C23, C24, C26, C28, C3, C4, C43, C57, C58, C59: footprint (none) -> Capacitor_SMD:C_0805_2012Metric
- C10, C11, C12, C13, C14, C15, C16, C17, C18, C19, C20, C21, C25, C27, C29, C30, C31, C32, C33, C34, C35, C39, C40, C41, C42, C44, C45, C46, C47, C48, C49, C5, C50, C51, C52, C53, C54, C55, C56, C6, C60, C7, C8, C9: footprint (none) -> Capacitor_SMD:C_0603_1608Metric
- C37: footprint (none) -> Capacitor_SMD:C_1812_4532Metric
- D1, Q1, Q2: footprint (none) -> Package_TO_SOT_SMD:SOT-23
- D2: footprint (none) -> Diode_SMD:D_0603_1608Metric
- D3: footprint (none) -> Diode_SMD:D_SOD-323
- D4: footprint (none) -> Diode_SMD:D_SOD-123
- FB1, FB2, L5, L6: footprint (none) -> Inductor_SMD:L_0603_1608Metric
- FL1: footprint (none) -> Inductor_SMD:L_CommonModeChoke_Coilank_ACM3216
- J1: footprint (none) -> Connector_JST:JST_GH_SM10B-GHS-TB_1x10-1MP_P1.25mm_Horizontal
- J2: footprint (none) -> Connector_JST:JST_GH_SM06B-GHS-TB_1x06-1MP_P1.25mm_Horizontal
- J3, J5: footprint (none) -> Connector_JST:JST_GH_SM04B-GHS-TB_1x04-1MP_P1.25mm_Horizontal
- J4, J6: footprint (none) -> Connector_JST:JST_GH_SM02B-GHS-TB_1x02-1MP_P1.25mm_Horizontal
- L1, L2: footprint (none) -> Inductor_SMD:L_1008_2520Metric
- L3, L4: footprint (none) -> Inductor_SMD:L_1210_3225Metric
- L7: footprint (none) -> Inductor_SMD:L_Coilcraft_XAL4030-XXX
- R1, R10, R17, R19, R2, R20, R21, R22, R23, R24, R25, R26, R27, R28, R3, R4, R5, R6, R7, R8, R9: footprint (none) -> Resistor_SMD:R_0603_1608Metric
- R18: footprint (none) -> Resistor_SMD:R_1206_3216Metric
- T2, T3: footprint (none) -> Triad:Triad_SP-74_THT_10.4x7.9mm_P2.54mm
- T4: footprint (none) -> Bourns:Bourns_SM-LP-5001_12.8x9.0mm_P2.54mm
- U1, U2: footprint (none) -> Package_SON:WSON-8-1EP_2x2mm_P0.5mm_EP0.9x1.6mm_ThermalVias
- U10, U11: footprint (none) -> Panasonic:Panasonic_GU-SOP8_4.4x9.37mm_P2.54mm_AQW61xS
- U12: footprint (none) -> Package_TO_SOT_SMD:SOT-23-5
- U3: footprint (none) -> Package_TO_SOT_SMD:TSOT-23-5
- U4: footprint (none) -> AnalogDevices:AD_LFCSP-88-1EP_12x12mm_P0.5mm_EP5.3x5.3mm_CP-88-10
- U5: footprint (none) -> Package_SO:SOIC-8_5.3x5.3mm_P1.27mm
- U6: footprint (none) -> AnalogDevices:AD_LFCSP-40-1EP_6x6mm_P0.5mm_EP4.3x4.3mm_CP-40-10
- U7: footprint (none) -> Infineon:Infineon_PG-TLGA-4-2_3.35x2.5mm_IM68A130A
- U9: footprint (none) -> Package_DFN_QFN:QFN-32-1EP_5x5mm_P0.5mm_EP3.6x3.6mm_ThermalVias
- Y1: footprint (none) -> Oscillator:Oscillator_SMD_SiT_PQFN-4Pin_3.2x2.5mm
