File: kicad/audio-board/boom-mic-tx-select.kicad_sch (KiCad schematic)
At the start: 15 parts, among them J4 BOOM_MIC_FROM_EARCUP, J5 TRS_TO_PJ068_AIRCRAFT, K1 G6K-2F-Y, Q1 2N7002, T1 SM-LP-5001, U11 ADP7118AUJZ-1.8-R7

Commit message: [LIMA] T1 isolates only the AeroNode leg - boom mic's bias loop to the aircraft must stay direct, per Peter
Peter: "bias will come from aircraft so DC must pass through to the
boom mic." Real correction to the architecture, not a tweak: T1
previously sat between K1's common and J5, isolating BOTH the
AeroNode injection path AND the boom-mic path from the aircraft.
That breaks the boom mic outright - the aircraft's electret bias
(8-16V, Bose A20 reference) rides as a complete DC loop through Tip
and Sleeve, and a transformer in that loop blocks it in every relay
state, not just while AeroNode is talking.

Fix: T1 now sits between C38 and K1.14 (NO_A) only - HPOUTP -> C38
-> T1 -> R13 -> K1.14. K1.11 (COM_A) wires directly to J5 Tip, no
transformer in the way. De-energized (boom mic mode), the path is
now fully direct and unisolated: aircraft bias flows Tip -> relay
contact -> J4.1 -> capsule -> J4.2 -> Sleeve -> aircraft, same as if
this board weren't in the circuit at all. Energized (AeroNode mode),
T1 still isolates AeroNode's own electronics from the aircraft -
the isolation goal survives, scoped to the leg that actually needs
it. J4 pin 2 changed from AGND to AC_GND to match - the boom mic
connector is electrically part of the aircraft's circuit now, not
AeroNode's, and its return has to complete the same aircraft-side
loop Sleeve does.

This closes the "boom mic gets no bias" open item from two commits
ago outright rather than carrying it forward - it was never a gap
needing a local bias supply, it was a routing mistake.

Caught a real short while rerouting: K1.11-to-J5-Tip auto-routed
through the exact point where J5's Sleeve/AC_GND stub landed,
shorting Tip to ground. find_shorted_nets caught it immediately;
a visual check would not have, since the two wires only touched at
one coordinate. Rerouted via a different corner. Same class of bug
as the collinear-wire shorts earlier in this sheet's history.

Verified: ERC errors unchanged at 46, 0 shorted nets, 0 ove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
Connections:
- net AC_GND: now also J4.2 (Pin_2)
- net AGND: no longer D1.2 (A), J4.2 (Pin_2), K1.A2, Q1.3 (D)
- net at T1.2 (AB): now also C38.2; no longer K1.11
- net at K1.14: now also R13.2; no longer C38.2
- net at J5.1 (Pin_1): now also K1.11; no longer R13.2
- net MIC_LINE: no longer names the net of R13.1, T1.4 (SB)
- new net: D1.2 (A), K1.A2, Q1.3 (D)

Commit message: [LIMA] add earphone/RX audio mute relay (K2), independent of TX relay, per Peter
Mutes the aircraft's incoming earphone/intercom audio (J5 Ring,
previously NC) on its way to the cup, driven by a new independent
GPIO_RLY_RX_MUTE_3V3 on J1 pin 8 - not shared with the boom-mic
relay's GPIO_RLY_TX_SEL_3V3, per Peter's explicit call.

Mute rather than sum, per Peter: docs/audio-board-decision-record.md
Decision A puts ANC in the earcup on its own codec, not on this
board, which removes H1's forcing reason (continuous ANC injection)
for summing instead of muting.

K2/Q2/D3/R14 mirror K1/Q1/D1/R10's exact pattern - same relay
(G6K-2F-Y), same low-side 2N7002 coil driver, same fail-passive
gate pulldown, same RLY_COIL_SUPPLY rail (U11, now shared by both
coils) and AC_GND domain (this path never crosses into AeroNode's
AGND side, so no transformer is needed here). Renamed the sheet
BOOM MIC / TX SELECT -> AIRCRAFT AUDIO I/O since it now hosts both
directions. Hit the same collinear-wire-into-AC_GND short as the
TX side's earlier SCAR, twice, wiring this up - documented in both
sheets' notes.

Co-Authored-By: Claude Sonnet 5 <noreply@anthropic.com>
Parts:
- added D3: 1N4148, symbol Diode:1N4148
- added J6: AUDIO_OUT_TO_CUP, symbol Connector_Generic:Conn_01x02
- added K2: G6K-2F-Y, symbol Relay:Relay_DPDT
- added Q2: 2N7002, symbol Transistor_FET:2N7002
- added R14: 100k, symbol Device:R
Connections:
- net AC_GND: now also J6.2 (Pin_2)
- net AGND: now also Q2.2 (S), R14.2
- net RLY_COIL_SUPPLY: now also D3.1 (K), K2.A1
- net at J5.2 (Pin_2): now also K2.12
- new net: J6.1 (Pin_1), K2.11
- new net: D3.2 (A), K2.A2, Q2.3 (D)
- new net GPIO_RLY_RX_MUTE_3V3: Q2.1 (G), R14.1
- no-connect marks 4 -> 7
Other:
- note added: "EARPHONE / RX AUDIO MUTE - added 2026-09-30, per Peter's question "should we use another relay to switch between audio coming from the aircraft to the cup and audio coming from the pi via the a2b or a summing arrangement?" This is the AIRCRAFT-TO-CUP direction (RX), separate from the TX circuit above (aircraft's mic input). WHY ON THIS SHEET: J5 (TRS_TO_PJ068_AIRCRAFT) already carries the aircraf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"
- note added: "TX AUDIO SELECT - relay switches what reaches the aircraft's mic jack between ADAU1861's own analog output (AeroNode speaking) and the pilot's boom mic (from the earcup), per Peter 2026-09-29. This sheet was renamed AIRCRAFT AUDIO I/O 2026-09-30 - it now also hosts the earphone/RX audio mute circuit (K2/J6/Q2/D3/R14), which reuses this sheet's J5 (Ring, previously NC) and RLY_COIL_SUPPLY. See the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"
- note removed: "TX AUDIO SELECT - relay switches what reaches the aircraft's mic jack between ADAU1861's own analog output (AeroNode speaking) and the pilot's boom mic (from the earcup), per Peter 2026-09-29. K1 = G6K-2F-Y (same qualified relay used on the H1 headset-mute board - bifurcated crossbar contacts, rated for dry-circuit audio, NOT a generic silver-contact relay). Only pole A is used; pole B (pins 21/2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"

Commit message: [LIMA] audio board: SP-74 per cup + AQW612S mic backup; cup T1 moved off, per Peter
Audio board, AIRCRAFT AUDIO I/O sheet:
- TX: relay K1 (+D1) replaced by AQW612S U12. N.C. = boom mic (J4.1) to
  aircraft Tip, so the pilot can still transmit unpowered; the aircraft's mic
  bias still flows DC-direct through it. N.O. = the existing T1/R13 injection
  path. Drive: 4.5 V (U11) -> R15 220R -> both LEDs in series -> Q1 low side
  (kept, with R10 pulldown): ~10 mA typ, >=6 mA worst case.
- RX: mute relay K2 (+Q2/D3/R14) removed. Two SP-74s (T2 left, T3 right),
  primaries in parallel on Ring/Sleeve, secondaries to J6/J7 for each cup.
  One per cup so a shorted cable can't silence both cups. GPIO_RLY_RX_MUTE_3V3
  removed (sheet pin, labels); J1 pin 8 spare, no-connect.
- Orphan no-connects and junctions from the relays removed; sheet notes
  rewritten (relay history: commits 6e258c8..e763f7c).

Cup board: T1 removed; J5 now receives the isolated secondary pair as
XF_SEC_A/XF_SEC_B (feeds U4/U5 N.C. and the ADC2 tap, unchanged).

Verified: audio-board ERC 45 errors (= baseline, all pre-existing main-sheet
unconnected pins), warnings 12 -> 11; netlist diff exactly as intended;
find_shorted_nets 0, overlaps 0, sheet pins valid; rendered. Cup board: ERC 0
errors / same 8 warnings, netlist diff exactly T1 out and J5 relabelled.
Note: kicad-cli did not register two plain pin-to-pin wires (R15-U12.1,
U12.2-U12.3) although their endpoints matched the pins exactly; replaced with
net labels (TX_SW_A, TX_SW_MID), after which all pins appear. Root cause not found.

Co-Authored-By: Claude Opus 5.5 <noreply@anthropic.com>
Parts:
- removed D1, D3: 1N4148, symbol Diode:1N4148
- removed K1, K2: G6K-2F-Y, symbol Relay:Relay_DPDT
- removed Q2: 2N7002, symbol Transistor_FET:2N7002
- removed R14: 100k, symbol Device:R
- added J7: AUDIO_OUT_TO_CUP_R, symbol Connector_Generic:Conn_01x02
- added R15: 220, symbol Device:R
- added T2, T3: SP-74, symbol Device:Transformer_1P_2S
- added U12: AQW612S, symbol Panasonic:AQW612S
- J6: value AUDIO_OUT_TO_CUP -> AUDIO_OUT_TO_CUP_L
Connections:
- net AC_GND: now also T2.2 (AB), T3.2 (AB); no longer J6.2 (Pin_2)
- net RLY_COIL_SUPPLY: now also R15.1
- net TX_SW_K: now reaches Q1.3 (D)
- net TX_SW_K: now also U12.4 (NO_LED_K)
- net TX_INJ: now reaches R13.2
- net TX_INJ: now also U12.5 (NO)
- net BOOM_MIC: now reaches J4.1 (Pin_1)
- net BOOM_MIC: now also U12.7 (NC)
- net MIC_TIP: now reaches J5.1 (Pin_1)
- net MIC_TIP: now also U12.6 (NO), U12.8 (NC)
- net XF_SEC_A_L: now reaches J6.1 (Pin_1)
- net XF_SEC_A_L: now also T2.3 (SA), T2.5 (SC)
- net RX_RING: now reaches J5.2 (Pin_2)
- net RX_RING: now also T2.1 (AA), T3.1 (AA)
- new net TX_SW_A: R15.2, U12.1 (NC_LED_A)
- new net TX_SW_MID: U12.2 (NC_LED_K), U12.3 (NO_LED_A)
- new net XF_SEC_A_R: J7.1 (Pin_1), T3.3 (SA), T3.5 (SC)
- new net XF_SEC_B_L: J6.2 (Pin_2), T2.4 (SB), T2.6 (SD)
- new net XF_SEC_B_R: J7.2 (Pin_2), T3.4 (SB), T3.6 (SD)
- no-connect marks 7 -> 0
Other:
- note added: "AIRCRAFT AUDIO I/O - rebuilt 2026-10-20, per Peter. Relays K1 (TX select) and K2 (RX mute) removed. History of the relay design: git log on this file (commits 6e258c8 .. e763f7c). J5 = aircraft TRS (PJ068 adapter): Tip = mic out to aircraft (MIC_TIP), Ring = earphone audio in (RX_RING), Sleeve = aircraft ground (AC_GND). TX - MIC TO AIRCRAFT, U12 (Panasonic AQW612S, 1 Form A + 1 Form B) - N.C. (7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"
- note removed: "EARPHONE / RX AUDIO MUTE - added 2026-09-30, per Peter's question "should we use another relay to switch between audio coming from the aircraft to the cup and audio coming from the pi via the a2b or a summing arrangement?" This is the AIRCRAFT-TO-CUP direction (RX), separate from the TX circuit above (aircraft's mic input). WHY ON THIS SHEET: J5 (TRS_TO_PJ068_AIRCRAFT) already carries the aircraf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"
- note removed: "TX AUDIO SELECT - relay switches what reaches the aircraft's mic jack between ADAU1861's own analog output (AeroNode speaking) and the pilot's boom mic (from the earcup), per Peter 2026-09-29. This sheet was renamed AIRCRAFT AUDIO I/O 2026-09-30 - it now also hosts the earphone/RX audio mute circuit (K2/J6/Q2/D3/R14), which reuses this sheet's J5 (Ring, previously NC) and RLY_COIL_SUPPLY. See the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"
