File: kicad/cup-board/cup-board.kicad_sch (KiCad schematic)
At the start: 29 parts, among them J2 EARCUP_SPKR, J3 CUP_PWR_IN, J4 VLED_IN, J5 AIRCRAFT_AUDIO_IN, J6 RLY_COIL_IN, K1 G6K-2F-Y DC5, T1 SP-74, U1 ADAU1861, U2 LSM6DSV16BX, U3 MAXM86161

Commit message: [LIMA] cup-board: T1 symbol swapped to Transformer_1P_2S, numbered as Triad SP-74
The old Device:Transformer_SP_2S had a centre tap and 7-pin numbering that did not
match the part. T1 is now Device:Transformer_1P_2S: 1 AC_AUDIO, 2 AC_GND, 3+5 XF_SEC_A,
4+6 XF_SEC_B (secondaries in parallel; dots on 1/3/5). The pin-2 no-connect flag is removed.

Verified: ERC 0 errors, same 8 pre-existing warnings; find_shorted_nets 0;
overlaps 0; kicad-cli netlist nets match. SVG re-exported.

Co-Authored-By: Claude Opus 5.5 <noreply@anthropic.com>
Parts:
- T1: symbol Device:Transformer_SP_2S -> Device:Transformer_1P_2S
Connections:
- net AC_GND: now also T1.2 (AB); no longer T1.3 (IN-)
- net XF_SEC_A: now also T1.3 (SA), T1.5 (SC); no longer T1.4 (OUT1A), T1.6 (OUT2A)
- net XF_SEC_B: now also T1.4 (SB), T1.6 (SD); no longer T1.5 (OUT1B), T1.7 (OUT2B)
- no-connect marks 37 -> 36
Changed lines of the file:
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@@
 		(at 314.96 231.14)
 	)
-	(no_connect
-		(at 88.9 228.6)
-	)
 	(wire
 		(pts
@@
 	(wire
 		(pts
-			(xy 88.9 223.52)
-			(xy 86.36 223.52)
-		)
-	)
-	(wire
-		(pts
-			(xy 88.9 233.68)
-			(xy 86.36 233.68)
-		)
-	)
-	(wire
-		(pts
-			(xy 109.22 218.44)
-			(xy 111.76 218.44)
-		)
-	)
-	(wire
-		(pts
-			(xy 109.22 226.06)
-			(xy 111.76 226.06)
-		)
-	)
-	(wire
-		(pts
-			(xy 109.22 231.14)
-			(xy 111.76 231.14)
-		)
-	)
-	(wire
-		(pts
-			(xy 109.22 238.76)
-			(xy 111.76 238.76)
-		)
-	)
-	(wire
-		(pts
 			(xy 118.11 185.42)
 			(xy 115.57 185.42)
@@
 		)
 	)
+	(wire
+		(pts
+			(xy 88.9 223.52)
+			(xy 86.36 223.52)
+		)
+	)
+	(wire
+		(pts
+			(xy 88.9 233.68)
+			(xy 86.36 233.68)
+		)
+	)
+	(wire
+		(pts
+			(xy 109.22 218.44)
+			(xy 111.76 218.44)
+		)
+	)
+	(wire
+		(pts
+			(xy 109.22 226.06)
+			(xy 111.76 226.06)
+		)
+	)
+	(wire
+		(pts
+			(xy 109.22 231.14)
+			(xy 111.76 231.14)
+		)
+	)
+	(wire
+		(pts
+			(xy 109.22 238.76)
+			(xy 111.76 238.76)
+		)
+	)
 	(label "1V8"
 		(at 160.02 82.55 0)
@@
 		)
 	)
-	(label "AC_AUDIO"
-		(at 86.36 223.52 180)
-		(effects
-			(font
-				(size 1.27 1.27)
-			)
-			(justify right bottom)
-		)
-	)
-	(label "AC_GND"
-		(at 86.36 233.68 180)
-		(effects
-			(font
-				(size 1.27 1.27)
-			)
-			(justify right bottom)
-		)
-	)
-	(label "XF_SEC_A"
-		(at 111.76 218.44 0)
-		(effects
-			(font
-				(size 1.27 1.27)
-			)
-			(justify left bottom)
-		)
-	)
-	(label "XF_SEC_B"
-		(at 111.76 226.06 0)
-		(effects
-			(font
-				(size 1.27 1.27)
-			)
-			(justify left bottom)
-		)
-	)
-	(label "XF_SEC_A"
-		(at 111.76 231.14 0)
-		(effects
-			(font
-				(size 1.27 1.27)
-			)
-			(justify left bottom)
-		)
-	)
-	(label "XF_SEC_B"
-		(at 111.76 238.76 0)
-		(effects
-			(font
-				(size 1.27 1.27)
-			)
-			(justify left bottom)
-		)
-	)
 	(label "XF_SEC_A"
 		(at 115.57 185.42 180)
@@
 		)
 	)
+	(label "AC_AUDIO"
+		(at 86.36 223.52 180)
+		(effects
+			(font
+				(size 1.27 1.27)
+			)
+			(justify right bottom)
+		)
+	)
+	(label "AC_GND"
+		(at 86.36 233.68 180)
+		(effects
+			(font
+				(size 1.27 1.27)
+			)
+			(justify right bottom)
+		)
+	)
+	(label "XF_SEC_A"
+		(at 111.76 218.44 0)
+		(effects
+			(font
+				(size 1.27 1.27)
+			)
+			(justify left bottom)
+		)
+	)
+	(label "XF_SEC_B"
+		(at 111.76 226.06 0)
+		(effects
+			(font
+				(size 1.27 1.27)
+			)
+			(justify left bottom)
+		)
+	)
+	(label "XF_SEC_A"
+		(at 111.76 231.14 0)
+		(effects
+			(font
+				(size 1.27 1.27)
+			)
+			(justify left bottom)
+		)
+	)
+	(label "XF_SEC_B"
+		(at 111.76 238.76 0)
+		(effects
+			(font
+				(size 1.27 1.27)
+			)
+			(justify left bottom)
+		)
+	)
 	(symbol
 		(lib_id "AnalogDevices:ADAU1861")
@@
 	)
 	(symbol
-		(lib_id "Device:Transformer_SP_2S")
+		(lib_id "Device:Transformer_1P_2S")
 		(at 99.06 228.6 0)
 		(unit 1)
